File: hardware/KiCAD/VolksEEG/ADS1299.sch (KiCad schematic (older format))
At the start: 1 part

Commit message: power supply finished
Connections:
- net VDDA: now reaches U?.19 (AVDD@1)
- net VDDA: now also U?.21 (AVDD@1), U?.22 (AVDD@1), U?.56 (AVDD@1), U?.59 (AVDD@2)
- net VSSA: now reaches U?.20 (AVSS@1)
- net VSSA: now also U?.23 (AVSS@1), U?.32 (AVSS@1), U?.57 (AVSS@1), U?.58 (AVSS@2)
- net GND: now reaches U?.33 (DGND)
- net GND: now also U?.49 (DGND), U?.51 (DGND)
- net +3V3: now reaches U?.48 (DVDD)
- net +3V3: now also U?.50 (DVDD)
Changed lines of the file:
@@
 Wire Wire Line
 	4150 2450 3500 2450
+Wire Wire Line
+	5550 1750 5550 1650
+Connection ~ 5550 1350
+Wire Wire Line
+	5550 1350 5700 1350
+Connection ~ 5550 1450
+Wire Wire Line
+	5550 1450 5550 1350
+Connection ~ 5550 1550
+Wire Wire Line
+	5550 1550 5550 1450
+Connection ~ 5550 1650
+Wire Wire Line
+	5550 1650 5550 1550
+Wire Wire Line
+	5550 5600 5550 5700
+Connection ~ 5550 5700
+Wire Wire Line
+	5550 5700 5550 5800
+Connection ~ 5550 5800
+Wire Wire Line
+	5550 5800 5550 5900
+Connection ~ 5550 5900
+Wire Wire Line
+	5550 5900 5550 6000
+$Comp
+L power:VSSA #PWR?
+U 1 1 615F7B61
+P 5650 6000
+F 0 "#PWR?" H 5650 5850 50  0001 C CNN
+F 1 "VSSA" V 5665 6128 50  0000 L CNN
+F 2 "" H 5650 6000 50  0001 C CNN
+F 3 "" H 5650 6000 50  0001 C CNN
+	1    5650 6000
+	0    1    1    0
+$EndComp
+Wire Wire Line
+	5650 6000 5550 6000
+Connection ~ 5550 6000
+$Comp
+L power:GND #PWR?
+U 1 1 615F94EE
+P 5650 6350
+AR Path="/615BA255/615F94EE" Ref="#PWR?"  Part="1"
+AR Path="/615BA110/615F94EE" Ref="#PWR?"  Part="1"
+F 0 "#PWR?" H 5650 6100 50  0001 C CNN
+F 1 "GND" H 5655 6177 50  0000 C CNN
+F 2 "" H 5650 6350 50  0001 C CNN
+F 3 "" H 5650 6350 50  0001 C CNN
+	1    5650 6350
+	0    -1   -1   0
+$EndComp
+Wire Wire Line
+	5650 6350 5550 6350
+Wire Wire Line
+	5550 6350 5550 6250
+Connection ~ 5550 6350
+Connection ~ 5550 6250
+Wire Wire Line
+	5550 6250 5550 6150
+Wire Wire Line
+	5550 2100 5550 2000
+$Comp
+L power:VDDA #PWR?
+U 1 1 615FCE43
+P 5700 1350
+F 0 "#PWR?" H 5700 1200 50  0001 C CNN
+F 1 "VDDA" V 5715 1478 50  0000 L CNN
+F 2 "" H 5700 1350 50  0001 C CNN
+F 3 "" H 5700 1350 50  0001 C CNN
+	1    5700 1350
+	0    1    1    0
+$EndComp
+$Comp
+L power:+3V3 #PWR?
+U 1 1 615FDD68
+P 5700 2000
+F 0 "#PWR?" H 5700 1850 50  0001 C CNN
+F 1 "+3V3" V 5715 2128 50  0000 L CNN
+F 2 "" H 5700 2000 50  0001 C CNN
+F 3 "" H 5700 2000 50  0001 C CNN
+	1    5700 2000
+	0    1    1    0
+$EndComp
+Wire Wire Line
+	5700 2000 5550 2000
+Connection ~ 5550 2000
 $EndSCHEMATC

Commit message: pcb layout update
Parts:
- gave numbers to parts that had none: 1
Changed lines of the file:
@@
 $EndDescr
 $Comp
-L VolksEEG:ADS1299IPAG U?
+L VolksEEG:ADS1299IPAG U1
 U 1 1 6161CDC0
 P 4850 3850
-F 0 "U?" H 4850 6620 50  0000 C CNN
+F 0 "U1" H 4850 6620 50  0000 C CNN
 F 1 "ADS1299IPAG" H 4850 6529 50  0000 C CNN
 F 2 "VolksEEG:QFP50P1200X1200X120-64N" H 4850 3850 50  0001 L BNN
@@
 	5550 5900 5550 6000
 $Comp
-L power:VSSA #PWR?
+L power:VSSA #PWR01
 U 1 1 615F7B61
 P 5650 6000
-F 0 "#PWR?" H 5650 5850 50  0001 C CNN
+F 0 "#PWR01" H 5650 5850 50  0001 C CNN
 F 1 "VSSA" V 5665 6128 50  0000 L CNN
 F 2 "" H 5650 6000 50  0001 C CNN
@@
 P 5650 6350
 AR Path="/615BA255/615F94EE" Ref="#PWR?"  Part="1"
-AR Path="/615BA110/615F94EE" Ref="#PWR?"  Part="1"
-F 0 "#PWR?" H 5650 6100 50  0001 C CNN
+AR Path="/615BA110/615F94EE" Ref="#PWR02"  Part="1"
+F 0 "#PWR02" H 5650 6100 50  0001 C CNN
 F 1 "GND" H 5655 6177 50  0000 C CNN
 F 2 "" H 5650 6350 50  0001 C CNN
@@
 	5550 2100 5550 2000
 $Comp
-L power:VDDA #PWR?
+L power:VDDA #PWR03
 U 1 1 615FCE43
 P 5700 1350
-F 0 "#PWR?" H 5700 1200 50  0001 C CNN
+F 0 "#PWR03" H 5700 1200 50  0001 C CNN
 F 1 "VDDA" V 5715 1478 50  0000 L CNN
 F 2 "" H 5700 1350 50  0001 C CNN
@@
 $EndComp
 $Comp
-L power:+3V3 #PWR?
+L power:+3V3 #PWR04
 U 1 1 615FDD68
 P 5700 2000
-F 0 "#PWR?" H 5700 1850 50  0001 C CNN
+F 0 "#PWR04" H 5700 1850 50  0001 C CNN
 F 1 "+3V3" V 5715 2128 50  0000 L CNN
 F 2 "" H 5700 2000 50  0001 C CNN

Commit message: Update
Parts:
- added C? (x5): 100n, symbol Device:C
- added C? (x9): 1u, symbol Device:C
- added C?: 100u, symbol Device:C
- added R?: 10k, symbol Device:R
- added U?: OPA388IDGKR, VolksEEG:SOP65P490X110-8N, symbol VolksEEG:OPA388IDGKR
Connections:
- net GND is gone; now on net GNDA: U1.33 (DGND), U1.49 (DGND), U1.51 (DGND)
- net +3V3: now also C?.1, C?.1, R?.1
- net ADS-nRST: now also R?.2
- net VDDA: now also U1.54 (AVDD1), C?.1, C?.1, C?.1, C?.1, C?.1, C?.1
- net VSSA: now also U1.53 (AVSS1), C?.1, C?.1, C?.2, C?.2, C?.2, C?.2, C?.2, C?.2, C?.2, C?.2, C?.2
- net at U1.26 (VCAP4): now also C?.1
- net at U1.28 (VCAP1): now also C?.1
- net at U1.30 (VCAP2): now also C?.1
- net GNDA: now reaches U1.31 (RESV1)
- net GNDA: now also U1.64 (RESERVED), C?.2, C?.2, C?.2, C?.2, C?.2, C?.2
- net at U1.55 (VCAP3): now also C?.1, C?.1
