File: hardware/KiCAD/VolksEEG/ADS1299.sch (KiCad schematic (older format))
At the start: 21 parts, among them U1 ADS1299IPAG

Commit message: Added debugging bits to more schematic sheets.
Connections:
- net GNDA: no longer C?.2, C?.2, J?.8 (Pin_8), U1.33 (DGND), U1.49 (DGND), U1.51 (DGND)
- new net GNDD: C?.2, C?.2, J?.8 (Pin_8), U1.33 (DGND), U1.49 (DGND), U1.51 (DGND)
Changed lines of the file:
@@
-$Comp
-L power:GNDA #PWR?
-U 1 1 617B92B5
-P 6150 6600
-F 0 "#PWR?" H 6150 6350 50  0001 C CNN
-F 1 "GNDA" H 6155 6427 50  0000 C CNN
-F 2 "" H 6150 6600 50  0001 C CNN
-F 3 "" H 6150 6600 50  0001 C CNN
-	1    6150 6600
-	1    0    0    -1
-$EndComp
 $Comp
 L power:GNDA #PWR?
@@
 Wire Bus Line
 	1750 5450 3700 5450
+$Comp
+L power:GNDD #PWR?
+U 1 1 618C346D
+P 6150 6600
+F 0 "#PWR?" H 6150 6350 50  0001 C CNN
+F 1 "GNDD" H 6154 6445 50  0000 C CNN
+F 2 "" H 6150 6600 50  0001 C CNN
+F 3 "" H 6150 6600 50  0001 C CNN
+	1    6150 6600
+	1    0    0    -1
+$EndComp
 $EndSCHEMATC

Commit message: tweaks to the ADS1299 schematic.
Parts:
- added R?: 10K, symbol Device:R
- R?: value ? -> 10K
Connections:
- net +3V3: now also R?.2
- net GNDA: now also C?.2, C?.2
- net GNDD: no longer C?.2, C?.2
- net nCS: now also R?.1
Changed lines of the file:
@@
 AIN8
 Wire Wire Line
-	3500 4250 4150 4250
+	3500 4250 3700 4250
 Wire Wire Line
 	3500 4350 4150 4350
@@
 Wire Wire Line
 	5550 6350 5550 6250
-Connection ~ 5550 6350
 Connection ~ 5550 6250
 Wire Wire Line
@@
 U 1 1 617D1100
 P 6650 2050
-F 0 "R?" V 6750 1950 50  0000 L CNN
-F 1 "?" V 6750 2100 50  0000 L CNN
+F 0 "R?" V 6750 2100 50  0000 L CNN
+F 1 "10K" V 6750 1900 50  0000 L CNN
 F 2 "" V 6580 2050 50  0001 C CNN
 F 3 "~" H 6650 2050 50  0001 C CNN
@@
 $EndComp
 Wire Wire Line
-	5550 6350 5800 6350
-Wire Wire Line
 	5800 6350 6150 6350
-Connection ~ 5800 6350
 Wire Wire Line
 	6150 6000 6150 6050
@@
 	5800 6000 6150 6000
 Wire Wire Line
-	6150 6600 6150 6500
-Connection ~ 6150 6350
+	5550 6600 5550 6500
 Wire Wire Line
 	6150 5950 6150 6000
@@
 GNDA
 Wire Wire Line
-	6550 6500 6150 6500
-Connection ~ 6150 6500
-Wire Wire Line
-	6150 6500 6150 6350
+	5650 6500 5550 6500
+Connection ~ 5550 6500
+Wire Wire Line
+	5550 6500 5550 6350
 $Comp
 L power:+2V5 #PWR?
@@
 	5700 2550 5850 2550
 Connection ~ 5700 2550
-Text HLabel 6550 6500 2    50   Input ~ 0
+Text HLabel 5650 6500 2    50   Input ~ 0
 GNDD
+$Comp
+L power:GNDD #PWR?
+U 1 1 618C346D
+P 5550 6600
+F 0 "#PWR?" H 5550 6350 50  0001 C CNN
+F 1 "GNDD" H 5554 6445 50  0000 C CNN
+F 2 "" H 5550 6600 50  0001 C CNN
+F 3 "" H 5550 6600 50  0001 C CNN
+	1    5550 6600
+	1    0    0    -1
+$EndComp
+Connection ~ 5550 6350
+$Comp
+L power:GNDA #PWR?
+U 1 1 619136C2
+P 6150 6450
+F 0 "#PWR?" H 6150 6200 50  0001 C CNN
+F 1 "GNDA" H 6155 6277 50  0000 C CNN
+F 2 "" H 6150 6450 50  0001 C CNN
+F 3 "" H 6150 6450 50  0001 C CNN
+	1    6150 6450
+	1    0    0    -1
+$EndComp
+Wire Wire Line
+	6150 6350 6150 6450
+Connection ~ 6150 6350
+$Comp
+L Device:R R?
+U 1 1 6191B069
+P 2900 4100
+F 0 "R?" H 2970 4146 50  0000 L CNN
+F 1 "10K" H 2970 4055 50  0000 L CNN
+F 2 "" V 2830 4100 50  0001 C CNN
+F 3 "~" H 2900 4100 50  0001 C CNN
+	1    2900 4100
+	0    1    1    0
+$EndComp
+$Comp
+L power:+3V3 #PWR?
+U 1 1 6191B9AF
+P 2500 4000
+F 0 "#PWR?" H 2500 3850 50  0001 C CNN
+F 1 "+3V3" H 2515 4173 50  0000 C CNN
+F 2 "" H 2500 4000 50  0001 C CNN
+F 3 "" H 2500 4000 50  0001 C CNN
+	1    2500 4000
+	1    0    0    -1
+$EndComp
+Wire Wire Line
+	2750 4100 2500 4100
+Wire Wire Line
+	2500 4100 2500 4000
+Wire Wire Line
+	3050 4100 3700 4100
+Wire Wire Line
+	3700 4100 3700 4250
 Wire Bus Line
 	1750 5450 3700 5450
-$Comp
-L power:GNDD #PWR?
-U 1 1 618C346D
-P 6150 6600
-F 0 "#PWR?" H 6150 6350 50  0001 C CNN
-F 1 "GNDD" H 6154 6445 50  0000 C CNN
-F 2 "" H 6150 6600 50  0001 C CNN
-F 3 "" H 6150 6600 50  0001 C CNN
-	1    6150 6600
-	1    0    0    -1
-$EndComp
+Connection ~ 3700 4250
+Wire Wire Line
+	3700 4250 4150 4250
 $EndSCHEMATC

Commit message: finished off tasks list.
Parts:
- removed J?: Conn_02x05_Counter_Clockwise, symbol Connector_Generic:Conn_02x05_Counter_Clockwise
- added J?: Conn_02x04_Counter_Clockwise, symbol Connector_Generic:Conn_02x04_Counter_Clockwise
- C?: value 1u -> 100n
- R?: value ? -> 10K
Connections:
- net GNDD is gone; now on net GNDA: U1.33 (DGND), U1.49 (DGND), U1.51 (DGND)
- net +2V5: now also J?.6 (Pin_6)
- net +3V3: now also J?.5 (Pin_5)
- net -2V5: now also J?.8 (Pin_8)
- net GNDA: now also J?.7 (Pin_7)
- net GPIO_1: now also J?.4 (Pin_4)
- net GPIO_2: now also J?.3 (Pin_3)
- net GPIO_3: now also J?.2 (Pin_2)
- net GPIO_4: now also J?.1 (Pin_1)
Changed lines of the file:
@@
 P 2050 4650
 F 0 "R?" H 2120 4696 50  0000 L CNN
-F 1 "?" H 2120 4605 50  0000 L CNN
+F 1 "10K" H 2120 4605 50  0000 L CNN
 F 2 "" V 1980 4650 50  0001 C CNN
 F 3 "~" H 2050 4650 50  0001 C CNN
@@
 	5900 800  5900 750
 Text HLabel 6900 1600 2    50   Input ~ 0
-+3V3
++3V3A
 Wire Wire Line
 	6900 1600 6650 1600
@@
 AR Path="/615BA255/61791774" Ref="C?"  Part="1"
 F 0 "C?" H 6265 6246 50  0000 L CNN
-F 1 "1u" H 6265 6155 50  0000 L CNN
+F 1 "100n" H 6265 6155 50  0000 L CNN
 F 2 "" H 6188 6050 50  0001 C CNN
 F 3 "~" H 6150 6200 50  0001 C CNN
@@
 Wire Wire Line
 	5800 6000 6150 6000
-Wire Wire Line
-	5550 6600 5550 6500
 Wire Wire Line
 	6150 5950 6150 6000
@@
 GPIO_4
 $Comp
-L power:+3V3 #PWR?
-U 1 1 61C79F8F
-P 3800 700
-F 0 "#PWR?" H 3800 550 50  0001 C CNN
-F 1 "+3V3" H 3815 873 50  0000 C CNN
-F 2 "" H 3800 700 50  0001 C CNN
-F 3 "" H 3800 700 50  0001 C CNN
-	1    3800 700
-	1    0    0    -1
-$EndComp
-$Comp
-L power:+3V3 #PWR?
-U 1 1 61C7A2A4
-P 6650 1500
-F 0 "#PWR?" H 6650 1350 50  0001 C CNN
-F 1 "+3V3" H 6665 1673 50  0000 C CNN
-F 2 "" H 6650 1500 50  0001 C CNN
-F 3 "" H 6650 1500 50  0001 C CNN
-	1    6650 1500
-	1    0    0    -1
-$EndComp
-$Comp
 L power:-2V5 #PWR?
 U 1 1 61C7B555
@@
 Text HLabel 5850 2550 2    50   Input ~ 0
 GNDA
-Wire Wire Line
-	5650 6500 5550 6500
-Connection ~ 5550 6500
-Wire Wire Line
-	5550 6500 5550 6350
 $Comp
 L power:+2V5 #PWR?
@@
 L power:-2V5 #PWR?
 U 1 1 61C87E18
-P 2050 6450
-F 0 "#PWR?" H 2050 6550 50  0001 C CNN
-F 1 "-2V5" H 2065 6623 50  0000 C CNN
-F 2 "" H 2050 6450 50  0001 C CNN
-F 3 "" H 2050 6450 50  0001 C CNN
-	1    2050 6450
+P 1950 6450
+F 0 "#PWR?" H 1950 6550 50  0001 C CNN
+F 1 "-2V5" H 1965 6623 50  0000 C CNN
+F 2 "" H 1950 6450 50  0001 C CNN
+F 3 "" H 1950 6450 50  0001 C CNN
+	1    1950 6450
 	-1   0    0    1
 $EndComp
@@
 L power:+2V5 #PWR?
 U 1 1 61C88C39
-P 1650 6700
-F 0 "#PWR?" H 1650 6550 50  0001 C CNN
-F 1 "+2V5" H 1665 6873 50  0000 C CNN
-F 2 "" H 1650 6700 50  0001 C CNN
-F 3 "" H 1650 6700 50  0001 C CNN
-	1    1650 6700
-	-1   0    0    1
-$EndComp
-$Comp
-L power:+3V3 #PWR?
-U 1 1 61C8974E
-P 1450 6450
-F 0 "#PWR?" H 1450 6300 50  0001 C CNN
-F 1 "+3V3" H 1465 6623 50  0000 C CNN
-F 2 "" H 1450 6450 50  0001 C CNN
-F 3 "" H 1450 6450 50  0001 C CNN
-	1    1450 6450
-	-1   0    0    1
-$EndComp
-$Comp
-L Connector_Generic:Conn_02x05_Counter_Clockwise J?
-U 1 1 61C8B3F1
-P 1750 6000
-F 0 "J?" V 1754 6280 50  0000 L CNN
-F 1 "Conn_02x05_Counter_Clockwise" V 1845 6280 50  0000 L CNN
-F 2 "" H 1750 6000 50  0001 C CNN
-F 3 "~" H 1750 6000 50  0001 C CNN
-	1    1750 6000
-	0    1    1    0
-$EndComp
-$Comp
-L power:GNDD #PWR?
-U 1 1 61C8E243
-P 1750 6450
-AR Path="/615BA20B/61C8E243" Ref="#PWR?"  Part="1"
-AR Path="/61731DC5/61C8E243" Ref="#PWR?"  Part="1"
-AR Path="/615BA255/61C8E243" Ref="#PWR?"  Part="1"
-AR Path="/615BA110/61C8E243" Ref="#PWR?"  Part="1"
-F 0 "#PWR?" H 1750 6200 50  0001 C CNN
-F 1 "GNDD" H 1754 6295 50  0000 C CNN
-F 2 "" H 1750 6450 50  0001 C CNN
-F 3 "" H 1750 6450 50  0001 C CNN
-	1    1750 6450
-	1    0    0    -1
-$EndComp
-Wire Wire Line
-	1450 6450 1450 6400
-Wire Wire Line
-	1450 6400 1550 6400
-Wire Wire Line
-	1550 6400 1550 6300
-Wire Wire Line
-	1950 6300 1950 6400
-Wire Wire Line
-	1950 6400 2050 6400
-Wire Wire Line
-	2050 6400 2050 6450
-Wire Wire Line
-	1750 6300 1750 6450
-Wire Wire Line
-	1650 6300 1650 6700
+P 1650 6650
+F 0 "#PWR?" H 1650 6500 50  0001 C CNN
+F 1 "+2V5" H 1665 6823 50  0000 C CNN
+F 2 "" H 1650 6650 50  0001 C CNN
+F 3 "" H 1650 6650 50  0001 C CNN
+	1    1650 6650
+	1    0    0    -1
+$EndComp
 Wire Wire Line
 	1850 6700 1850 6300
@@
 	5700 2550 5850 2550
 Connection ~ 5700 2550
-Text HLabel 5650 6500 2    50   Input ~ 0
-GNDD
-$Comp
-L power:GNDD #PWR?
-U 1 1 618C346D
-P 5550 6600
-F 0 "#PWR?" H 5550 6350 50  0001 C CNN
-F 1 "GNDD" H 5554 6445 50  0000 C CNN
-F 2 "" H 5550 6600 50  0001 C CNN
-F 3 "" H 5550 6600 50  0001 C CNN
-	1    5550 6600
-	1    0    0    -1
-$EndComp
-Connection ~ 5550 6350
 $Comp
 L power:GNDA #PWR?
@@
 	0    1    1    0
 $EndComp
-$Comp
-L power:+3V3 #PWR?
-U 1 1 6191B9AF
+Wire Wire Line
+	2750 4100 2500 4100
+Wire Wire Line
+	2500 4100 2500 4000
+Wire Wire Line
+	3050 4100 3700 4100
+Wire Wire Line
+	3700 4100 3700 4250
+Connection ~ 3700 4250
+Wire Wire Line
+	3700 4250 4150 4250
+Wire Wire Line
+	5550 6350 5800 6350
+Connection ~ 5550 6350
+Connection ~ 5800 6350
+$Comp
+L VolksEEG:+3V3A #PWR?
+U 1 1 619467FC
+P 3800 700
+AR Path="/615BA255/619467FC" Ref="#PWR?"  Part="1"
+AR Path="/615BA110/619467FC" Ref="#PWR?"  Part="1"
+F 0 "#PWR?" H 3800 550 50  0001 C CNN
+F 1 "+3V3A" H 3815 873 50  0000 C CNN
+F 2 "" H 3800 700 50  0001 C CNN
+F 3 "" H 3800 700 50  0001 C CNN
+	1    3800 700
+	1    0    0    -1
+$EndComp
+$Comp
+L VolksEEG:+3V3A #PWR?
+U 1 1 6194CA89
+P 6650 1500
+AR Path="/615BA255/6194CA89" Ref="#PWR?"  Part="1"
+AR Path="/615BA110/6194CA89" Ref="#PWR?"  Part="1"
+F 0 "#PWR?" H 6650 1350 50  0001 C CNN
+F 1 "+3V3A" H 6665 1673 50  0000 C CNN
+F 2 "" H 6650 1500 50  0001 C CNN
+F 3 "" H 6650 1500 50  0001 C CNN
+	1    6650 1500
+	1    0    0    -1
+$EndComp
+$Comp
+L VolksEEG:+3V3A #PWR?
+U 1 1 61952D7C
 P 2500 4000
+AR Path="/615BA255/61952D7C" Ref="#PWR?"  Part="1"
+AR Path="/615BA110/61952D7C" Ref="#PWR?"  Part="1"
 F 0 "#PWR?" H 2500 3850 50  0001 C CNN
-F 1 "+3V3" H 2515 4173 50  0000 C CNN
+F 1 "+3V3A" H 2515 4173 50  0000 C CNN
 F 2 "" H 2500 4000 50  0001 C CNN
 F 3 "" H 2500 4000 50  0001 C CNN
@@
 	1    0    0    -1
 $EndComp
-Wire Wire Line
-	2750 4100 2500 4100
-Wire Wire Line
-	2500 4100 2500 4000
-Wire Wire Line
-	3050 4100 3700 4100
-Wire Wire Line
-	3700 4100 3700 4250
+$Comp
+L VolksEEG:+3V3A #PWR?
+U 1 1 61959043
+P 1400 6350
+AR Path="/615BA255/61959043" Ref="#PWR?"  Part="1"
+AR Path="/615BA110/61959043" Ref="#PWR?"  Part="1"
+F 0 "#PWR?" H 1400 6200 50  0001 C CNN
+F 1 "+3V3A" H 1415 6523 50  0000 C CNN
+F 2 "" H 1400 6350 50  0001 C CNN
+F 3 "" H 1400 6350 50  0001 C CNN
+	1    1400 6350
+	1    0    0    -1
+$EndComp
+$Comp
+L Connector_Generic:Conn_02x04_Counter_Clockwise J?
+U 1 1 61960524
+P 1850 6000
+F 0 "J?" V 1854 6180 50  0000 L CNN
+F 1 "Conn_02x04_Counter_Clockwise" V 1945 6180 50  0000 L CNN
+F 2 "" H 1850 6000 50  0001 C CNN
+F 3 "~" H 1850 6000 50  0001 C CNN
+	1    1850 6000
+	0    1    1    0
+$EndComp
+Wire Wire Line
+	1950 6300 1950 6450
+Wire Wire Line
+	1650 6300 1650 6400
+Wire Wire Line
+	1650 6400 1400 6400
+Wire Wire Line
+	1400 6400 1400 6350
+Wire Wire Line
+	1650 6700 1750 6700
+Wire Wire Line
+	1750 6700 1750 6300
+Wire Wire Line
+	1650 6700 1650 6650
 Wire Bus Line
 	1750 5450 3700 5450
-Connection ~ 3700 4250
-Wire Wire Line
-	3700 4250 4150 4250
 $EndSCHEMATC
