File: hardware/KiCAD/VolksEEG/EEG-Electrodes.sch (KiCad schematic (older format))
At the start: 21 parts, among them J4 Conn_01x10

Commit message: Updated some footprints and part manufacturers and numbers.
Parts:
- C10: Manufacturer (none) -> KYOCERA AVX; Part Number (none) -> 08055A152FAT2A
- C11, C12, C13, C14, C15, C7, C8, C9: footprint Capacitor_SMD:C_0603_1608Metric_Pad1.08x0.95mm_HandSolder -> Capacitor_SMD:C_0805_2012Metric_Pad1.18x1.45mm_HandSolder; Manufacturer (none) -> KEMET; Part Number (none) -> C0805C333F3GEC7210
- J4: footprint (none) -> Connector_PinHeader_2.54mm:PinHeader_1x10_P2.54mm_Vertical; Manufacturer (none) -> TE Connectivity AMP Connectors; Part Number (none) -> 1-640456-0
Changed lines of the file:
@@
 F 0 "C7" H 2615 4396 50  0000 L CNN
 F 1 "33n" H 2615 4305 50  0000 L CNN
-F 2 "Capacitor_SMD:C_0603_1608Metric_Pad1.08x0.95mm_HandSolder" H 2538 4200 50  0001 C CNN
+F 2 "Capacitor_SMD:C_0805_2012Metric_Pad1.18x1.45mm_HandSolder" H 2538 4200 50  0001 C CNN
 F 3 "~" H 2500 4350 50  0001 C CNN
+F 4 "KEMET" H 2500 4350 50  0001 C CNN "Manufacturer"
+F 5 "C0805C333F3GEC7210" H 2500 4350 50  0001 C CNN "Part Number"
 	1    2500 4350
 	1    0    0    -1
@@
 F 0 "C8" H 3015 4396 50  0000 L CNN
 F 1 "33n" H 3015 4305 50  0000 L CNN
-F 2 "Capacitor_SMD:C_0603_1608Metric_Pad1.08x0.95mm_HandSolder" H 2938 4200 50  0001 C CNN
+F 2 "Capacitor_SMD:C_0805_2012Metric_Pad1.18x1.45mm_HandSolder" H 2938 4200 50  0001 C CNN
 F 3 "~" H 2900 4350 50  0001 C CNN
+F 4 "KEMET" H 2900 4350 50  0001 C CNN "Manufacturer"
+F 5 "C0805C333F3GEC7210" H 2900 4350 50  0001 C CNN "Part Number"
 	1    2900 4350
 	1    0    0    -1
@@
 F 0 "C9" H 3415 4396 50  0000 L CNN
 F 1 "33n" H 3415 4305 50  0000 L CNN
-F 2 "Capacitor_SMD:C_0603_1608Metric_Pad1.08x0.95mm_HandSolder" H 3338 4200 50  0001 C CNN
+F 2 "Capacitor_SMD:C_0805_2012Metric_Pad1.18x1.45mm_HandSolder" H 3338 4200 50  0001 C CNN
 F 3 "~" H 3300 4350 50  0001 C CNN
+F 4 "KEMET" H 3300 4350 50  0001 C CNN "Manufacturer"
+F 5 "C0805C333F3GEC7210" H 3300 4350 50  0001 C CNN "Part Number"
 	1    3300 4350
 	1    0    0    -1
@@
 F 0 "C11" H 3815 4396 50  0000 L CNN
 F 1 "33n" H 3815 4305 50  0000 L CNN
-F 2 "Capacitor_SMD:C_0603_1608Metric_Pad1.08x0.95mm_HandSolder" H 3738 4200 50  0001 C CNN
+F 2 "Capacitor_SMD:C_0805_2012Metric_Pad1.18x1.45mm_HandSolder" H 3738 4200 50  0001 C CNN
 F 3 "~" H 3700 4350 50  0001 C CNN
+F 4 "KEMET" H 3700 4350 50  0001 C CNN "Manufacturer"
+F 5 "C0805C333F3GEC7210" H 3700 4350 50  0001 C CNN "Part Number"
 	1    3700 4350
 	1    0    0    -1
@@
 F 0 "C12" H 4215 4396 50  0000 L CNN
 F 1 "33n" H 4215 4305 50  0000 L CNN
-F 2 "Capacitor_SMD:C_0603_1608Metric_Pad1.08x0.95mm_HandSolder" H 4138 4200 50  0001 C CNN
+F 2 "Capacitor_SMD:C_0805_2012Metric_Pad1.18x1.45mm_HandSolder" H 4138 4200 50  0001 C CNN
 F 3 "~" H 4100 4350 50  0001 C CNN
+F 4 "KEMET" H 4100 4350 50  0001 C CNN "Manufacturer"
+F 5 "C0805C333F3GEC7210" H 4100 4350 50  0001 C CNN "Part Number"
 	1    4100 4350
 	1    0    0    -1
@@
 F 0 "C13" H 4615 4396 50  0000 L CNN
 F 1 "33n" H 4615 4305 50  0000 L CNN
-F 2 "Capacitor_SMD:C_0603_1608Metric_Pad1.08x0.95mm_HandSolder" H 4538 4200 50  0001 C CNN
+F 2 "Capacitor_SMD:C_0805_2012Metric_Pad1.18x1.45mm_HandSolder" H 4538 4200 50  0001 C CNN
 F 3 "~" H 4500 4350 50  0001 C CNN
+F 4 "KEMET" H 4500 4350 50  0001 C CNN "Manufacturer"
+F 5 "C0805C333F3GEC7210" H 4500 4350 50  0001 C CNN "Part Number"
 	1    4500 4350
 	1    0    0    -1
@@
 F 0 "C14" H 5065 4396 50  0000 L CNN
 F 1 "33n" H 5065 4305 50  0000 L CNN
-F 2 "Capacitor_SMD:C_0603_1608Metric_Pad1.08x0.95mm_HandSolder" H 4988 4200 50  0001 C CNN
+F 2 "Capacitor_SMD:C_0805_2012Metric_Pad1.18x1.45mm_HandSolder" H 4988 4200 50  0001 C CNN
 F 3 "~" H 4950 4350 50  0001 C CNN
+F 4 "KEMET" H 4950 4350 50  0001 C CNN "Manufacturer"
+F 5 "C0805C333F3GEC7210" H 4950 4350 50  0001 C CNN "Part Number"
 	1    4950 4350
 	1    0    0    -1
@@
 F 0 "C15" H 5465 4396 50  0000 L CNN
 F 1 "33n" H 5465 4305 50  0000 L CNN
-F 2 "Capacitor_SMD:C_0603_1608Metric_Pad1.08x0.95mm_HandSolder" H 5388 4200 50  0001 C CNN
+F 2 "Capacitor_SMD:C_0805_2012Metric_Pad1.18x1.45mm_HandSolder" H 5388 4200 50  0001 C CNN
 F 3 "~" H 5350 4350 50  0001 C CNN
+F 4 "KEMET" H 5350 4350 50  0001 C CNN "Manufacturer"
+F 5 "C0805C333F3GEC7210" H 5350 4350 50  0001 C CNN "Part Number"
 	1    5350 4350
 	1    0    0    -1
@@
 F 2 "Capacitor_SMD:C_0603_1608Metric_Pad1.08x0.95mm_HandSolder" H 3338 4900 50  0001 C CNN
 F 3 "~" H 3300 5050 50  0001 C CNN
+F 4 "KYOCERA AVX" H 3300 5050 50  0001 C CNN "Manufacturer"
+F 5 "08055A152FAT2A" H 3300 5050 50  0001 C CNN "Part Number"
 	1    3300 5050
 	-1   0    0    1
@@
 F 0 "J4" H 8580 3142 50  0000 L CNN
 F 1 "Conn_01x10" H 8580 3051 50  0000 L CNN
-F 2 "" H 8500 3150 50  0001 C CNN
+F 2 "Connector_PinHeader_2.54mm:PinHeader_1x10_P2.54mm_Vertical" H 8500 3150 50  0001 C CNN
 F 3 "~" H 8500 3150 50  0001 C CNN
+F 4 "TE Connectivity AMP Connectors" H 8500 3150 50  0001 C CNN "Manufacturer"
+F 5 "1-640456-0" H 8500 3150 50  0001 C CNN "Part Number"
 	1    8500 3150
 	1    0    0    -1

Commit message: Finished adding footprints, and started laying out the isolation section.
Parts:
- R20: Manufacturer (none) -> TE Connectivity Passive Product; Part Number (none) -> CPF0603B1M0E1
- R21, R22, R23, R24, R25, R26, R27, R28, R29, R30: Manufacturer (none) -> Stackpole Electronics Inc; Part Number (none) -> RNCF0603TKY4K99
Changed lines of the file:
@@
 F 2 "Resistor_SMD:R_0603_1608Metric_Pad0.98x0.95mm_HandSolder" V 5730 1850 50  0001 C CNN
 F 3 "~" H 5800 1850 50  0001 C CNN
+F 4 "Stackpole Electronics Inc" H 5800 1850 50  0001 C CNN "Manufacturer"
+F 5 "RNCF0603TKY4K99" H 5800 1850 50  0001 C CNN "Part Number"
 	1    5800 1850
 	0    1    1    0
@@
 F 2 "Resistor_SMD:R_0603_1608Metric_Pad0.98x0.95mm_HandSolder" V 5730 2150 50  0001 C CNN
 F 3 "~" H 5800 2150 50  0001 C CNN
+F 4 "Stackpole Electronics Inc" H 5800 2150 50  0001 C CNN "Manufacturer"
+F 5 "RNCF0603TKY4K99" H 5800 2150 50  0001 C CNN "Part Number"
 	1    5800 2150
 	0    1    1    0
@@
 F 2 "Resistor_SMD:R_0603_1608Metric_Pad0.98x0.95mm_HandSolder" V 5730 2450 50  0001 C CNN
 F 3 "~" H 5800 2450 50  0001 C CNN
+F 4 "Stackpole Electronics Inc" H 5800 2450 50  0001 C CNN "Manufacturer"
+F 5 "RNCF0603TKY4K99" H 5800 2450 50  0001 C CNN "Part Number"
 	1    5800 2450
 	0    1    1    0
@@
 F 2 "Resistor_SMD:R_0603_1608Metric_Pad0.98x0.95mm_HandSolder" V 5730 3050 50  0001 C CNN
 F 3 "~" H 5800 3050 50  0001 C CNN
+F 4 "Stackpole Electronics Inc" H 5800 3050 50  0001 C CNN "Manufacturer"
+F 5 "RNCF0603TKY4K99" H 5800 3050 50  0001 C CNN "Part Number"
 	1    5800 3050
 	0    1    1    0
@@
 F 2 "Resistor_SMD:R_0603_1608Metric_Pad0.98x0.95mm_HandSolder" V 5730 2750 50  0001 C CNN
 F 3 "~" H 5800 2750 50  0001 C CNN
+F 4 "Stackpole Electronics Inc" H 5800 2750 50  0001 C CNN "Manufacturer"
+F 5 "RNCF0603TKY4K99" H 5800 2750 50  0001 C CNN "Part Number"
 	1    5800 2750
 	0    1    1    0
@@
 F 2 "Resistor_SMD:R_0603_1608Metric_Pad0.98x0.95mm_HandSolder" V 5730 3350 50  0001 C CNN
 F 3 "~" H 5800 3350 50  0001 C CNN
+F 4 "Stackpole Electronics Inc" H 5800 3350 50  0001 C CNN "Manufacturer"
+F 5 "RNCF0603TKY4K99" H 5800 3350 50  0001 C CNN "Part Number"
 	1    5800 3350
 	0    1    1    0
@@
 F 2 "Resistor_SMD:R_0603_1608Metric_Pad0.98x0.95mm_HandSolder" V 5730 3650 50  0001 C CNN
 F 3 "~" H 5800 3650 50  0001 C CNN
+F 4 "Stackpole Electronics Inc" H 5800 3650 50  0001 C CNN "Manufacturer"
+F 5 "RNCF0603TKY4K99" H 5800 3650 50  0001 C CNN "Part Number"
 	1    5800 3650
 	0    1    1    0
@@
 F 2 "Resistor_SMD:R_0603_1608Metric_Pad0.98x0.95mm_HandSolder" V 5730 3950 50  0001 C CNN
 F 3 "~" H 5800 3950 50  0001 C CNN
+F 4 "Stackpole Electronics Inc" H 5800 3950 50  0001 C CNN "Manufacturer"
+F 5 "RNCF0603TKY4K99" H 5800 3950 50  0001 C CNN "Part Number"
 	1    5800 3950
 	0    1    1    0
@@
 F 2 "Resistor_SMD:R_0603_1608Metric_Pad0.98x0.95mm_HandSolder" V 5730 4600 50  0001 C CNN
 F 3 "~" H 5800 4600 50  0001 C CNN
+F 4 "Stackpole Electronics Inc" H 5800 4600 50  0001 C CNN "Manufacturer"
+F 5 "RNCF0603TKY4K99" H 5800 4600 50  0001 C CNN "Part Number"
 	1    5800 4600
 	0    1    1    0
@@
 F 2 "Resistor_SMD:R_0603_1608Metric_Pad0.98x0.95mm_HandSolder" V 2830 5050 50  0001 C CNN
 F 3 "~" H 2900 5050 50  0001 C CNN
+F 4 "TE Connectivity Passive Product" H 2900 5050 50  0001 C CNN "Manufacturer"
+F 5 "CPF0603B1M0E1" H 2900 5050 50  0001 C CNN "Part Number"
 	1    2900 5050
 	1    0    0    -1
@@
 F 2 "Resistor_SMD:R_0603_1608Metric_Pad0.98x0.95mm_HandSolder" V 5730 5200 50  0001 C CNN
 F 3 "~" H 5800 5200 50  0001 C CNN
+F 4 "Stackpole Electronics Inc" H 5800 5200 50  0001 C CNN "Manufacturer"
+F 5 "RNCF0603TKY4K99" H 5800 5200 50  0001 C CNN "Part Number"
 	1    5800 5200
 	0    1    1    0
