File: hardware/KiCAD/VolksEEG/VolksEEG.sch (KiCad schematic (older format))
At the start: 0 parts

Commit message: power supply finished
Changed lines of the file:
@@
 F0 "nRF52840" 50
 F1 "nRF52840.sch" 50
-F2 "MOSI" O L 7300 3500 50
-F3 "SCK" O L 7300 3400 50
-F4 "MISO" I L 7300 3600 50
-F5 "nCS" O L 7300 3700 50
-F6 "ADS-nRST" O L 7300 3900 50
+F2 "MOSI" O L 7300 3450 50
+F3 "SCK" O L 7300 3350 50
+F4 "MISO" I L 7300 3550 50
+F5 "nCS" O L 7300 3650 50
+F6 "ADS-nRST" O L 7300 3850 50
 $EndSheet
 $Sheet
@@
 F17 "AIN8P" O R 4500 5350 50
 $EndSheet
+Wire Wire Line
+	4500 3500 5500 3500
+Wire Wire Line
+	5500 3600 4500 3600
+Wire Wire Line
+	4500 3750 5500 3750
+Wire Wire Line
+	5500 3850 4500 3850
+Wire Wire Line
+	4500 4000 5500 4000
+Wire Wire Line
+	5500 4100 4500 4100
+Wire Wire Line
+	4500 4250 5500 4250
+Wire Wire Line
+	5500 4350 4500 4350
+Wire Wire Line
+	4500 4500 5500 4500
+Wire Wire Line
+	5500 4600 4500 4600
+Wire Wire Line
+	4500 4750 5500 4750
+Wire Wire Line
+	5500 4850 4500 4850
+Wire Wire Line
+	4500 5000 5500 5000
+Wire Wire Line
+	5500 5100 4500 5100
+Wire Wire Line
+	4500 5250 5500 5250
+Wire Wire Line
+	5500 5350 4500 5350
+Wire Wire Line
+	6550 3350 7300 3350
+Wire Wire Line
+	7300 3450 6550 3450
+Wire Wire Line
+	6550 3550 7300 3550
+Wire Wire Line
+	7300 3650 6550 3650
+Wire Wire Line
+	6550 3850 7300 3850
 $EndSCHEMATC

Commit message: Update
Parts:
- added U7: ISO7761DW, Package_SO:SOIC-16W_7.5x10.3mm_P1.27mm, symbol Isolator:ISO7761DW
Connections:
- net ADS1299/ADS-nRST: now also U7.14 (OUTB)
- net ADS1299/MISO: now also U7.10 (INF)
- net ADS1299/MOSI: now also U7.15 (OUTA)
- net ADS1299/SCK: now also U7.12 (OUTD)
- net ADS1299/nCS: now also U7.13 (OUTC)
- new net +3V3: U7.16 (Vcc2)
- new net GNDA: U7.9 (GND2)
- new net GNDD: U7.8 (GND1)
- new net VDC: U7.1 (Vcc1)
- new net nRF52840/ADS-nRST: U7.3 (INB)
- new net nRF52840/MISO: U7.7 (OUTF)
- new net nRF52840/MOSI: U7.2 (INA)
- new net nRF52840/SCK: U7.5 (IND)
- new net nRF52840/nCS0: U7.4 (INC)
- no-connect marks 0 -> 2
Changed lines of the file:
@@
 F1 "ADS1299.sch" 50
 F2 "nCS" I R 6550 3650 50
-F3 "SCK" I R 6550 3350 50
+F3 "SCK" I R 6550 3750 50
 F4 "MOSI" I R 6550 3450 50
-F5 "MISO" O R 6550 3550 50
-F6 "ADS-nRST" I R 6550 3850 50
+F5 "MISO" O R 6550 3950 50
+F6 "ADS-nRST" I R 6550 3550 50
 F7 "AIN5N" I L 5500 4500 50
 F8 "AIN5P" I L 5500 4600 50
@@
 F21 "AIN4N" I L 5500 4250 50
 F22 "AIN4P" I L 5500 4350 50
-$EndSheet
-$Sheet
-S 7300 3150 1200 1300
-U 615BA20B
-F0 "nRF52840" 50
-F1 "nRF52840.sch" 50
-F2 "MOSI" O L 7300 3450 50
-F3 "SCK" O L 7300 3350 50
-F4 "MISO" I L 7300 3550 50
-F5 "nCS" O L 7300 3650 50
-F6 "ADS-nRST" O L 7300 3850 50
 $EndSheet
 $Sheet
@@
 Wire Wire Line
 	5500 5350 4500 5350
+$Sheet
+S 8850 3150 1200 1400
+U 615BA20B
+F0 "nRF52840" 50
+F1 "nRF52840.sch" 50
+F2 "MOSI" O L 8850 3450 50
+F3 "SCK" O L 8850 3750 50
+F4 "MISO" I L 8850 3950 50
+F5 "ADS-nRST" O L 8850 3550 50
+F6 "nCS0" O L 8850 3650 50
+$EndSheet
 Wire Wire Line
-	6550 3350 7300 3350
+	7300 3950 6550 3950
 Wire Wire Line
-	7300 3450 6550 3450
+	6550 3450 7300 3450
+Wire Wire Line
+	7300 3750 6550 3750
+Wire Wire Line
+	6550 3650 7300 3650
+Wire Wire Line
+	8850 3950 8100 3950
+Wire Wire Line
+	8100 3450 8850 3450
+Wire Wire Line
+	8850 3750 8100 3750
+Wire Wire Line
+	8100 3650 8850 3650
+$Comp
+L Isolator:ISO7761DW U7
+U 1 1 616504E1
+P 7700 3750
+F 0 "U7" H 7300 4350 50  0000 C CNN
+F 1 "ISO7761DW" H 7150 4250 50  0000 C CNN
+F 2 "Package_SO:SOIC-16W_7.5x10.3mm_P1.27mm" H 7925 3200 50  0001 L CNN
+F 3 "https://www.ti.com/lit/ds/symlink/iso7763.pdf" H 8100 3650 50  0001 C CNN
+	1    7700 3750
+	-1   0    0    -1
+$EndComp
+Wire Wire Line
+	8100 3550 8850 3550
 Wire Wire Line
 	6550 3550 7300 3550
-Wire Wire Line
-	7300 3650 6550 3650
-Wire Wire Line
-	6550 3850 7300 3850
+NoConn ~ 8100 3850
+NoConn ~ 7300 3850
+$Comp
+L power:GNDA #PWR?
+U 1 1 6181B798
+P 7500 4350
+AR Path="/615BA110/6181B798" Ref="#PWR?"  Part="1"
+AR Path="/6181B798" Ref="#PWR?"  Part="1"
+F 0 "#PWR?" H 7500 4100 50  0001 C CNN
+F 1 "GNDA" H 7505 4177 50  0000 C CNN
+F 2 "" H 7500 4350 50  0001 C CNN
+F 3 "" H 7500 4350 50  0001 C CNN
+	1    7500 4350
+	1    0    0    -1
+$EndComp
+$Comp
+L power:GNDD #PWR?
+U 1 1 6181F021
+P 7900 4350
+F 0 "#PWR?" H 7900 4100 50  0001 C CNN
+F 1 "GNDD" H 7904 4195 50  0000 C CNN
+F 2 "" H 7900 4350 50  0001 C CNN
+F 3 "" H 7900 4350 50  0001 C CNN
+	1    7900 4350
+	1    0    0    -1
+$EndComp
+$Comp
+L power:VDC #PWR?
+U 1 1 6181F86F
+P 7900 3050
+F 0 "#PWR?" H 7900 2950 50  0001 C CNN
+F 1 "VDC" H 7915 3223 50  0000 C CNN
+F 2 "" H 7900 3050 50  0001 C CNN
+F 3 "" H 7900 3050 50  0001 C CNN
+	1    7900 3050
+	1    0    0    -1
+$EndComp
+$Comp
+L power:+3V3 #PWR?
+U 1 1 6181FC38
+P 7500 3050
+F 0 "#PWR?" H 7500 2900 50  0001 C CNN
+F 1 "+3V3" H 7515 3223 50  0000 C CNN
+F 2 "" H 7500 3050 50  0001 C CNN
+F 3 "" H 7500 3050 50  0001 C CNN
+	1    7500 3050
+	1    0    0    -1
+$EndComp
 $EndSCHEMATC
