File: hardware/KiCAD/VolksEEG/_autosave-ADS1299.sch (KiCad schematic (older format))
At the start: 18 parts, among them U1 ADS1299IPAG

Commit message: Update
Connections:
- net VDDA: now also U1.54 (AVDD1)
- net VSSA: now also U1.53 (AVSS1)
Other:
- moved on the sheet: U?
Changed lines of the file:
@@
 L VolksEEG:OPA388IDGKR U?
 U 1 1 617AA68D
-P 8650 3600
-F 0 "U?" H 8994 3646 50  0000 L CNN
-F 1 "OPA388IDGKR" H 8994 3555 50  0000 L CNN
-F 2 "VolksEEG:SOP65P490X110-8N" H 8650 3600 50  0001 C CNN
-F 3 "https://www.ti.com/lit/gpn/opa388" H 8650 3600 50  0001 C CNN
-	1    8650 3600
+P 7650 3450
+F 0 "U?" H 7994 3496 50  0000 L CNN
+F 1 "OPA388IDGKR" H 7994 3405 50  0000 L CNN
+F 2 "VolksEEG:SOP65P490X110-8N" H 7650 3450 50  0001 C CNN
+F 3 "https://www.ti.com/lit/gpn/opa388" H 7650 3450 50  0001 C CNN
+	1    7650 3450
 	1    0    0    -1
 $EndComp
@@
 	0    1    1    0
 $EndComp
+Wire Wire Line
+	5550 1850 5550 1750
+Connection ~ 5550 1750
+Wire Wire Line
+	5550 5450 5550 5600
+Connection ~ 5550 5600
 $EndSCHEMATC
