File: hardware/KiCAD/VolksEEG/nRF52840.sch (KiCad schematic (older format))
At the start: 30 parts, among them J1 Conn_01x03, J2 QWIIC, J3 693061010911, U1 nRF52840-Feather-Sense-Board

Commit message: Updated some footprints and part manufacturers and numbers.
Parts:
- C1: Manufacturer (none) -> Samsung Electro-Mechanics; Part Number (none) -> CL21B104KACNNNC
- D1: footprint (none) -> LED_SMD:LED_0603_1608Metric_Pad1.05x0.95mm_HandSolder; Manufacturer (none) -> Stanley Electric Co; Part Number (none) -> VFHR1111C-3BY2A-TR
- J1: footprint (none) -> Connector_PinHeader_2.54mm:PinHeader_1x03_P2.54mm_Vertical; Manufacturer (none) -> TE Connectivity AMP Connectors; Part Number (none) -> 640456-3
- J2: footprint (none) -> Connector_PinHeader_2.54mm:PinHeader_1x04_P2.54mm_Vertical; Manufacturer (none) -> TE Connectivity AMP Connectors; Part Number (none) -> 640456-4
- J3: Manufacturer (none) -> Würth Elektronik; Part Number (none) -> 693061010911
- R3: value 220R -> 1K; Manufacturer (none) -> Stackpole Electronics Inc; Part Number (none) -> RMCF0603FG1K00
- TP1, TP2, TP3, TP4, TP5, TP6, TP7: footprint (none) -> TestPoint:TestPoint_Keystone_5010-5014_Multipurpose; Manufacturer (none) -> N/A; Part Number (none) -> N/A
- TP31: footprint (none) -> TestPoint:TestPoint_Bridge_Pitch7.62mm_Drill1.3mm; Manufacturer (none) -> N/A; Part Number (none) -> N/A
Other:
- note added: "Footprint is not correct."
Changed lines of the file:
@@
 F 0 "J2" H 8428 5546 50  0000 L CNN
 F 1 "QWIIC" H 8428 5455 50  0000 L CNN
-F 2 "" H 8250 5500 50  0001 C CNN
+F 2 "Connector_PinHeader_2.54mm:PinHeader_1x04_P2.54mm_Vertical" H 8250 5500 50  0001 C CNN
 F 3 "" H 8250 5500 50  0001 C CNN
+F 4 "TE Connectivity AMP Connectors" H 8250 5500 50  0001 C CNN "Manufacturer"
+F 5 "640456-4" H 8250 5500 50  0001 C CNN "Part Number"
 	1    8250 5500
 	1    0    0    -1
@@
 F 0 "J1" H 8230 4642 50  0000 L CNN
 F 1 "Conn_01x03" H 8230 4551 50  0000 L CNN
-F 2 "" H 8150 4600 50  0001 C CNN
+F 2 "Connector_PinHeader_2.54mm:PinHeader_1x03_P2.54mm_Vertical" H 8150 4600 50  0001 C CNN
 F 3 "~" H 8150 4600 50  0001 C CNN
+F 4 "TE Connectivity AMP Connectors" H 8150 4600 50  0001 C CNN "Manufacturer"
+F 5 "640456-3" H 8150 4600 50  0001 C CNN "Part Number"
 	1    8150 4600
 	1    0    0    -1
@@
 F 2 "Capacitor_SMD:C_0603_1608Metric_Pad1.08x0.95mm_HandSolder" H 8038 1850 50  0001 C CNN
 F 3 "~" H 8000 2000 50  0001 C CNN
+F 4 "Samsung Electro-Mechanics" H 8000 2000 50  0001 C CNN "Manufacturer"
+F 5 "CL21B104KACNNNC" H 8000 2000 50  0001 C CNN "Part Number"
 	1    8000 2000
 	-1   0    0    1
@@
 F 2 "VolksEEG:693061010911" H 9600 1850 50  0001 L BNN
 F 3 "https://www.we-online.com/catalog/datasheet/693061010911.pdf" H 9600 1850 50  0001 L BNN
+F 4 "Würth Elektronik" H 9600 1850 50  0001 C CNN "Manufacturer"
+F 5 "693061010911" H 9600 1850 50  0001 C CNN "Part Number"
 	1    9600 1850
 	1    0    0    -1
@@
 F 0 "TP5" H 7058 5518 50  0000 L CNN
 F 1 "TestPoint" H 7058 5427 50  0001 L CNN
-F 2 "" H 7200 5400 50  0001 C CNN
+F 2 "TestPoint:TestPoint_Keystone_5010-5014_Multipurpose" H 7200 5400 50  0001 C CNN
 F 3 "~" H 7200 5400 50  0001 C CNN
+F 4 "N/A" H 7000 5400 50  0001 C CNN "Manufacturer"
+F 5 "N/A" H 7000 5400 50  0001 C CNN "Part Number"
 	1    7000 5400
 	1    0    0    -1
@@
 F 0 "TP4" H 6858 5268 50  0000 L CNN
 F 1 "TestPoint" H 6858 5177 50  0001 L CNN
-F 2 "" H 7000 5150 50  0001 C CNN
+F 2 "TestPoint:TestPoint_Keystone_5010-5014_Multipurpose" H 7000 5150 50  0001 C CNN
 F 3 "~" H 7000 5150 50  0001 C CNN
+F 4 "N/A" H 6800 5150 50  0001 C CNN "Manufacturer"
+F 5 "N/A" H 6800 5150 50  0001 C CNN "Part Number"
 	1    6800 5150
 	1    0    0    -1
@@
 F 0 "TP7" H 7908 4468 50  0000 L CNN
 F 1 "TestPoint" H 7908 4377 50  0001 L CNN
-F 2 "" H 8050 4350 50  0001 C CNN
+F 2 "TestPoint:TestPoint_Keystone_5010-5014_Multipurpose" H 8050 4350 50  0001 C CNN
 F 3 "~" H 8050 4350 50  0001 C CNN
+F 4 "N/A" H 7850 4350 50  0001 C CNN "Manufacturer"
+F 5 "N/A" H 7850 4350 50  0001 C CNN "Part Number"
 	1    7850 4350
 	1    0    0    -1
@@
 F 0 "TP6" H 7558 4218 50  0000 L CNN
 F 1 "TestPoint" H 7558 4127 50  0001 L CNN
-F 2 "" H 7700 4100 50  0001 C CNN
+F 2 "TestPoint:TestPoint_Keystone_5010-5014_Multipurpose" H 7700 4100 50  0001 C CNN
 F 3 "~" H 7700 4100 50  0001 C CNN
+F 4 "N/A" H 7500 4100 50  0001 C CNN "Manufacturer"
+F 5 "N/A" H 7500 4100 50  0001 C CNN "Part Number"
 	1    7500 4100
 	1    0    0    -1
@@
 F 0 "TP3" H 2008 4218 50  0000 L CNN
 F 1 "TestPoint" H 2008 4127 50  0001 L CNN
-F 2 "" H 2150 4100 50  0001 C CNN
+F 2 "TestPoint:TestPoint_Keystone_5010-5014_Multipurpose" H 2150 4100 50  0001 C CNN
 F 3 "~" H 2150 4100 50  0001 C CNN
+F 4 "N/A" H 1950 4100 50  0001 C CNN "Manufacturer"
+F 5 "N/A" H 1950 4100 50  0001 C CNN "Part Number"
 	1    1950 4100
 	1    0    0    -1
@@
 F 0 "TP2" H 1908 4018 50  0000 L CNN
 F 1 "TestPoint" H 1908 3927 50  0001 L CNN
-F 2 "" H 2050 3900 50  0001 C CNN
+F 2 "TestPoint:TestPoint_Keystone_5010-5014_Multipurpose" H 2050 3900 50  0001 C CNN
 F 3 "~" H 2050 3900 50  0001 C CNN
+F 4 "N/A" H 1850 3900 50  0001 C CNN "Manufacturer"
+F 5 "N/A" H 1850 3900 50  0001 C CNN "Part Number"
 	1    1850 3900
 	1    0    0    -1
@@
 F 0 "TP1" H 1808 3818 50  0000 L CNN
 F 1 "TestPoint" H 1808 3727 50  0001 L CNN
-F 2 "" H 1950 3700 50  0001 C CNN
+F 2 "TestPoint:TestPoint_Keystone_5010-5014_Multipurpose" H 1950 3700 50  0001 C CNN
 F 3 "~" H 1950 3700 50  0001 C CNN
+F 4 "N/A" H 1750 3700 50  0001 C CNN "Manufacturer"
+F 5 "N/A" H 1750 3700 50  0001 C CNN "Part Number"
 	1    1750 3700
 	1    0    0    -1
@@
 F 0 "D1" V 2250 1150 50  0000 C CNN
 F 1 "Red" V 2350 1200 50  0000 R CNN
-F 2 "" H 2300 1300 50  0001 C CNN
-F 3 "~" H 2300 1300 50  0001 C CNN
+F 2 "LED_SMD:LED_0603_1608Metric_Pad1.05x0.95mm_HandSolder" H 2300 1300 50  0001 C CNN
+F 3 "http://www.stanley-components.com/php/downloaddatafile.php?rp=0,VFHR1111C-3BY2A-TR_e.pdf" H 2300 1300 50  0001 C CNN
+F 4 "Stanley Electric Co" V 2300 1300 50  0001 C CNN "Manufacturer"
+F 5 "VFHR1111C-3BY2A-TR" V 2300 1300 50  0001 C CNN "Part Number"
 	1    2300 1300
 	0    -1   -1   0
@@
 P 2300 1750
 F 0 "R3" H 2150 1800 50  0000 C CNN
-F 1 "220R" H 2100 1700 50  0000 C CNN
+F 1 "1K" H 2100 1700 50  0000 C CNN
 F 2 "Resistor_SMD:R_0603_1608Metric_Pad0.98x0.95mm_HandSolder" V 2230 1750 50  0001 C CNN
-F 3 "~" H 2300 1750 50  0001 C CNN
+F 3 "https://www.seielect.com/catalog/sei-rmcf_rmcp.pdf" H 2300 1750 50  0001 C CNN
+F 4 "Stackpole Electronics Inc" H 2300 1750 50  0001 C CNN "Manufacturer"
+F 5 "RMCF0603FG1K00" H 2300 1750 50  0001 C CNN "Part Number"
 	1    2300 1750
 	-1   0    0    1
@@
 F 0 "TP31" H 5758 5218 50  0000 L CNN
 F 1 "TestPoint" H 5758 5127 50  0001 L CNN
-F 2 "" H 5900 5100 50  0001 C CNN
+F 2 "TestPoint:TestPoint_Bridge_Pitch7.62mm_Drill1.3mm" H 5900 5100 50  0001 C CNN
 F 3 "~" H 5900 5100 50  0001 C CNN
+F 4 "N/A" H 5700 5100 50  0001 C CNN "Manufacturer"
+F 5 "N/A" H 5700 5100 50  0001 C CNN "Part Number"
 	1    5700 5100
 	0    1    1    0
@@
 Wire Wire Line
 	8350 1750 9100 1750
+Text Notes 8100 5150 0    50   ~ 0
+Footprint is not correct.
 $EndSCHEMATC

Commit message: Finished adding footprints, and started laying out the isolation section.
Parts:
- R1, R14, R15, R16, R2, R4, R5, R6, R7: Manufacturer (none) -> Rohm Semiconductor; Part Number (none) -> TRR03EZPJ000
- R10, R11, R12, R8, R9: Manufacturer (none) -> Stackpole Electronics Inc; Part Number (none) -> RMCF0603FT4K70
- R17: footprint Resistor_SMD:R_0603_1608Metric_Pad0.98x0.95mm_HandSolder -> VolksEEG:high_power_chip_resistor; Manufacturer (none) -> TE Connectivity Passive Product; Part Number (none) -> 35502R2JT
- U1: Manufacturer (none) -> adafruit; Part Number (none) -> 4516
Changed lines of the file:
@@
 F 2 "Resistor_SMD:R_0603_1608Metric_Pad0.98x0.95mm_HandSolder" V 3730 4050 50  0001 C CNN
 F 3 "~" H 3800 4050 50  0001 C CNN
+F 4 "Stackpole Electronics Inc" H 3800 4050 50  0001 C CNN "Manufacturer"
+F 5 "RMCF0603FT4K70" H 3800 4050 50  0001 C CNN "Part Number"
 	1    3800 4050
 	1    0    0    -1
@@
 F 2 "Resistor_SMD:R_0603_1608Metric_Pad0.98x0.95mm_HandSolder" V 4030 4050 50  0001 C CNN
 F 3 "~" H 4100 4050 50  0001 C CNN
+F 4 "Stackpole Electronics Inc" H 4100 4050 50  0001 C CNN "Manufacturer"
+F 5 "RMCF0603FT4K70" H 4100 4050 50  0001 C CNN "Part Number"
 	1    4100 4050
 	1    0    0    -1
@@
 F 2 "Resistor_SMD:R_0603_1608Metric_Pad0.98x0.95mm_HandSolder" V 3430 4050 50  0001 C CNN
 F 3 "~" H 3500 4050 50  0001 C CNN
+F 4 "Stackpole Electronics Inc" H 3500 4050 50  0001 C CNN "Manufacturer"
+F 5 "RMCF0603FT4K70" H 3500 4050 50  0001 C CNN "Part Number"
 	1    3500 4050
 	1    0    0    -1
@@
 F 2 "Resistor_SMD:R_0603_1608Metric_Pad0.98x0.95mm_HandSolder" V 3130 4050 50  0001 C CNN
 F 3 "~" H 3200 4050 50  0001 C CNN
+F 4 "Stackpole Electronics Inc" H 3200 4050 50  0001 C CNN "Manufacturer"
+F 5 "RMCF0603FT4K70" H 3200 4050 50  0001 C CNN "Part Number"
 	1    3200 4050
 	1    0    0    -1
@@
 F 2 "Resistor_SMD:R_0603_1608Metric_Pad0.98x0.95mm_HandSolder" V 2830 4050 50  0001 C CNN
 F 3 "~" H 2900 4050 50  0001 C CNN
+F 4 "Stackpole Electronics Inc" H 2900 4050 50  0001 C CNN "Manufacturer"
+F 5 "RMCF0603FT4K70" H 2900 4050 50  0001 C CNN "Part Number"
 	1    2900 4050
 	1    0    0    -1
@@
 F 2 "Resistor_SMD:R_0603_1608Metric_Pad0.98x0.95mm_HandSolder" V 6330 4100 50  0001 C CNN
 F 3 "~" H 6400 4100 50  0001 C CNN
+F 4 "Rohm Semiconductor" H 6400 4100 50  0001 C CNN "Manufacturer"
+F 5 "TRR03EZPJ000" H 6400 4100 50  0001 C CNN "Part Number"
 	1    6400 4100
 	0    1    1    0
@@
 F 2 "Resistor_SMD:R_0603_1608Metric_Pad0.98x0.95mm_HandSolder" V 6580 4200 50  0001 C CNN
 F 3 "~" H 6650 4200 50  0001 C CNN
+F 4 "Rohm Semiconductor" H 6650 4200 50  0001 C CNN "Manufacturer"
+F 5 "TRR03EZPJ000" H 6650 4200 50  0001 C CNN "Part Number"
 	1    6650 4200
 	0    1    1    0
@@
 F 2 "Resistor_SMD:R_0603_1608Metric_Pad0.98x0.95mm_HandSolder" V 2580 4400 50  0001 C CNN
 F 3 "~" H 2650 4400 50  0001 C CNN
+F 4 "Rohm Semiconductor" H 2650 4400 50  0001 C CNN "Manufacturer"
+F 5 "TRR03EZPJ000" H 2650 4400 50  0001 C CNN "Part Number"
 	1    2650 4400
 	0    1    1    0
@@
 F 2 "Resistor_SMD:R_0603_1608Metric_Pad0.98x0.95mm_HandSolder" V 2330 4500 50  0001 C CNN
 F 3 "~" H 2400 4500 50  0001 C CNN
+F 4 "Rohm Semiconductor" H 2400 4500 50  0001 C CNN "Manufacturer"
+F 5 "TRR03EZPJ000" H 2400 4500 50  0001 C CNN "Part Number"
 	1    2400 4500
 	0    1    1    0
@@
 F 2 "Resistor_SMD:R_0603_1608Metric_Pad0.98x0.95mm_HandSolder" V 2080 4600 50  0001 C CNN
 F 3 "~" H 2150 4600 50  0001 C CNN
+F 4 "Rohm Semiconductor" H 2150 4600 50  0001 C CNN "Manufacturer"
+F 5 "TRR03EZPJ000" H 2150 4600 50  0001 C CNN "Part Number"
 	1    2150 4600
 	0    1    1    0
@@
 F 2 "Resistor_SMD:R_0603_1608Metric_Pad0.98x0.95mm_HandSolder" V 2580 4700 50  0001 C CNN
 F 3 "~" H 2650 4700 50  0001 C CNN
+F 4 "Rohm Semiconductor" H 2650 4700 50  0001 C CNN "Manufacturer"
+F 5 "TRR03EZPJ000" H 2650 4700 50  0001 C CNN "Part Number"
 	1    2650 4700
 	0    1    1    0
@@
 F 2 "Resistor_SMD:R_0603_1608Metric_Pad0.98x0.95mm_HandSolder" V 2330 4800 50  0001 C CNN
 F 3 "~" H 2400 4800 50  0001 C CNN
+F 4 "Rohm Semiconductor" H 2400 4800 50  0001 C CNN "Manufacturer"
+F 5 "TRR03EZPJ000" H 2400 4800 50  0001 C CNN "Part Number"
 	1    2400 4800
 	0    1    1    0
@@
 F 2 "Resistor_SMD:R_0603_1608Metric_Pad0.98x0.95mm_HandSolder" V 6080 4000 50  0001 C CNN
 F 3 "~" H 6150 4000 50  0001 C CNN
+F 4 "Rohm Semiconductor" H 6150 4000 50  0001 C CNN "Manufacturer"
+F 5 "TRR03EZPJ000" H 6150 4000 50  0001 C CNN "Part Number"
 	1    6150 4000
 	0    1    1    0
@@
 F 2 "Resistor_SMD:R_0603_1608Metric_Pad0.98x0.95mm_HandSolder" V 2080 4900 50  0001 C CNN
 F 3 "~" H 2150 4900 50  0001 C CNN
+F 4 "Rohm Semiconductor" H 2150 4900 50  0001 C CNN "Manufacturer"
+F 5 "TRR03EZPJ000" H 2150 4900 50  0001 C CNN "Part Number"
 	1    2150 4900
 	0    1    1    0
@@
 F 0 "R17" V 7793 1550 50  0000 C CNN
 F 1 "2R2" V 7884 1550 50  0000 C CNN
-F 2 "Resistor_SMD:R_0603_1608Metric_Pad0.98x0.95mm_HandSolder" V 7930 1550 50  0001 C CNN
+F 2 "VolksEEG:high_power_chip_resistor" V 7930 1550 50  0001 C CNN
 F 3 "~" H 8000 1550 50  0001 C CNN
+F 4 "TE Connectivity Passive Product" H 8000 1550 50  0001 C CNN "Manufacturer"
+F 5 "35502R2JT" H 8000 1550 50  0001 C CNN "Part Number"
 	1    8000 1550
 	-1   0    0    1
@@
 F 2 "VolksEEG:nRF52840_Feather_Sense" H 4550 5250 50  0001 C CNN
 F 3 "https://cdn-learn.adafruit.com/downloads/pdf/adafruit-feather-sense.pdf" H 4550 5250 50  0001 C CNN
+F 4 "adafruit" H 4900 4250 50  0001 C CNN "Manufacturer"
+F 5 "4516" H 4900 4250 50  0001 C CNN "Part Number"
 	1    4900 4250
 	1    0    0    -1

Commit message: Layout of the NRF52840 section of the PCB.
Connections:
- net MISO_ni: no longer R14.2, U1.13 (MISO)
- net MOSI_ni: no longer R15.2, U1.12 (MOSI)
- net SCK_ni: no longer R16.2, U1.11 (SCK)
- net SD-nCD_ni: now also R4.2, TP2.1; no longer R6.2, TP1.1
- net SD-nCS_ni: now also R6.2, TP1.1; no longer R1.2, TP3.1
- net SD-nWP_ni: now also R1.2, TP3.1; no longer R4.2, TP2.1
- net at R7.1, R9.2, U1.22 (10): no longer R8.2
- net at R5.1, U1.23 (11): now also R8.2
- new net: R16.2, U1.11 (SCK)
- new net: R15.2, U1.12 (MOSI)
- new net: R14.2, U1.13 (MISO)
Other:
- moved on the sheet: R14, R15, R16
Changed lines of the file:
@@
 ADS-nRST_ni
 Wire Wire Line
-	5400 4000 6000 4000
-Wire Wire Line
-	6900 4100 6550 4100
-Wire Wire Line
-	5400 4200 6500 4200
+	5400 4000 5550 4000
 NoConn ~ 4400 3450
 NoConn ~ 4400 3600
@@
 Text HLabel 1700 4900 0    50   Input ~ 0
 ADS-nDRDY_ni
-Text Label 1700 4400 2    50   ~ 0
+Text Label 1700 4500 2    50   ~ 0
 SD-nCD_ni
 Text HLabel 6150 3400 2    50   Output ~ 0
@@
 	1    0    0    -1
 $EndComp
-Text Label 1700 4600 2    50   ~ 0
+Text Label 1700 4400 2    50   ~ 0
 SD-nCS_ni
 $Comp
@@
 	1    0    0    -1
 $EndComp
-Text Label 5650 4000 0    50   ~ 0
+Text Label 6450 4000 0    50   ~ 0
 MISO_ni
-Text Label 5650 4100 0    50   ~ 0
+Text Label 6450 4100 0    50   ~ 0
 MOSI_ni
-Text Label 5650 4200 0    50   ~ 0
+Text Label 6450 4200 0    50   ~ 0
 SCK_ni
 Wire Wire Line
@@
 	2900 3800 3200 3800
 Connection ~ 3200 3800
-Text Label 1700 4500 2    50   ~ 0
+Text Label 1700 4600 2    50   ~ 0
 SD-nWP_ni
-Wire Wire Line
-	6300 4000 6900 4000
 $Comp
 L Device:R R15
 U 1 1 61DF07C8
-P 6400 4100
-F 0 "R15" V 6100 4100 50  0000 C CNN
-F 1 "0R" V 6200 4100 50  0000 C CNN
-F 2 "Resistor_SMD:R_0603_1608Metric_Pad0.98x0.95mm_HandSolder" V 6330 4100 50  0001 C CNN
-F 3 "~" H 6400 4100 50  0001 C CNN
-F 4 "Rohm Semiconductor" H 6400 4100 50  0001 C CNN "Manufacturer"
-F 5 "TRR03EZPJ000" H 6400 4100 50  0001 C CNN "Part Number"
-	1    6400 4100
-	0    1    1    0
-$EndComp
-Wire Wire Line
-	6250 4100 5400 4100
-$Comp
-L Device:R R16
-U 1 1 61DF0A54
-P 6650 4200
-F 0 "R16" V 6250 4200 50  0000 C CNN
-F 1 "0R" V 6350 4200 50  0000 C CNN
-F 2 "Resistor_SMD:R_0603_1608Metric_Pad0.98x0.95mm_HandSolder" V 6580 4200 50  0001 C CNN
-F 3 "~" H 6650 4200 50  0001 C CNN
-F 4 "Rohm Semiconductor" H 6650 4200 50  0001 C CNN "Manufacturer"
-F 5 "TRR03EZPJ000" H 6650 4200 50  0001 C CNN "Part Number"
-	1    6650 4200
-	0    1    1    0
-$EndComp
-Wire Wire Line
-	6800 4200 6900 4200
+P 5950 4100
+F 0 "R15" V 5650 4100 50  0000 C CNN
+F 1 "0R" V 5750 4100 50  0000 C CNN
+F 2 "Resistor_SMD:R_0603_1608Metric_Pad0.98x0.95mm_HandSolder" V 5880 4100 50  0001 C CNN
+F 3 "~" H 5950 4100 50  0001 C CNN
+F 4 "Rohm Semiconductor" H 5950 4100 50  0001 C CNN "Manufacturer"
+F 5 "TRR03EZPJ000" H 5950 4100 50  0001 C CNN "Part Number"
+	1    5950 4100
+	0    1    1    0
+$EndComp
 Wire Wire Line
 	1700 4600 1950 4600
@@
 Wire Wire Line
 	3200 4700 4400 4700
-Wire Wire Line
-	2900 4200 2900 4700
-Connection ~ 2900 4700
-Wire Wire Line
-	2900 4700 3200 4700
 $Comp
 L Device:R R6
@@
 	0    1    1    0
 $EndComp
-Wire Wire Line
-	2800 4700 2900 4700
 $Comp
 L Device:R R5
@@
 $EndComp
 Wire Wire Line
-	2550 4800 4400 4800
+	2550 4800 2900 4800
 $Comp
 L Device:R R14
 U 1 1 61DF0030
-P 6150 4000
-F 0 "R14" V 5943 4000 50  0000 C CNN
-F 1 "0R" V 6034 4000 50  0000 C CNN
-F 2 "Resistor_SMD:R_0603_1608Metric_Pad0.98x0.95mm_HandSolder" V 6080 4000 50  0001 C CNN
-F 3 "~" H 6150 4000 50  0001 C CNN
-F 4 "Rohm Semiconductor" H 6150 4000 50  0001 C CNN "Manufacturer"
-F 5 "TRR03EZPJ000" H 6150 4000 50  0001 C CNN "Part Number"
-	1    6150 4000
+P 5700 4000
+F 0 "R14" V 5493 4000 50  0000 C CNN
+F 1 "0R" V 5584 4000 50  0000 C CNN
+F 2 "Resistor_SMD:R_0603_1608Metric_Pad0.98x0.95mm_HandSolder" V 5630 4000 50  0001 C CNN
+F 3 "~" H 5700 4000 50  0001 C CNN
+F 4 "Rohm Semiconductor" H 5700 4000 50  0001 C CNN "Manufacturer"
+F 5 "TRR03EZPJ000" H 5700 4000 50  0001 C CNN "Part Number"
+	1    5700 4000
 	0    1    1    0
 $EndComp
@@
 Text Notes 8100 5150 0    50   ~ 0
 Footprint is not correct.
+Wire Wire Line
+	5850 4000 6900 4000
+Wire Wire Line
+	6100 4100 6900 4100
+$Comp
+L Device:R R16
+U 1 1 61DF0A54
+P 6200 4200
+F 0 "R16" V 5800 4200 50  0000 C CNN
+F 1 "0R" V 5900 4200 50  0000 C CNN
+F 2 "Resistor_SMD:R_0603_1608Metric_Pad0.98x0.95mm_HandSolder" V 6130 4200 50  0001 C CNN
+F 3 "~" H 6200 4200 50  0001 C CNN
+F 4 "Rohm Semiconductor" H 6200 4200 50  0001 C CNN "Manufacturer"
+F 5 "TRR03EZPJ000" H 6200 4200 50  0001 C CNN "Part Number"
+	1    6200 4200
+	0    1    1    0
+$EndComp
+Wire Wire Line
+	5400 4200 6050 4200
+Wire Wire Line
+	5400 4100 5800 4100
+Wire Wire Line
+	6350 4200 6900 4200
+Wire Notes Line
+	5550 3700 6850 3700
+Wire Notes Line
+	6850 3700 6850 4300
+Wire Notes Line
+	6850 4300 5550 4300
+Wire Notes Line
+	5550 4300 5550 3700
+Wire Wire Line
+	2800 4700 3200 4700
+Wire Wire Line
+	2900 4200 2900 4800
+Connection ~ 2900 4800
+Wire Wire Line
+	2900 4800 4400 4800
+Wire Notes Line
+	1200 4250 1800 4250
+Wire Notes Line
+	1800 4250 1800 4650
+Wire Notes Line
+	1800 4650 1200 4650
+Wire Notes Line
+	1200 4650 1200 4250
 $EndSCHEMATC
