File: hardware/KiCAD/VolksEEG/isolation.sch (KiCad schematic (older format))
At the start: 30 parts, among them U2 ADUM240E1BRIZ-RL, U3 ADUM240E1BRIZ-RL, U4 MEJ1S0305SC

Commit message: Change ADS1299 over to using the KiCAD library footprint.
Also deleted the custom drawn QFP footprint.
Parts:
- added JP5: Jumper_NC_Small, symbol Device:Jumper_NC_Small
- gave numbers to parts that had none: 2
Connections:
- wire segments 99 -> 97
Changed lines of the file:
@@
 Comment4 ""
 $EndDescr
-Text HLabel 7750 2000 0    50   Input ~ 0
+Text HLabel 7250 2000 0    50   Input ~ 0
 +3V3_ni
 Text HLabel 2000 2450 0    50   Input ~ 0
@@
 Text HLabel 5600 2750 2    50   Output ~ 0
 SCK
-Text HLabel 9950 2300 2    50   Output ~ 0
-GNDD
-Wire Wire Line
-	9950 2300 9850 2300
 $Comp
 L power:GNDD #PWR?
@@
 L Connector:TestPoint TP23
 U 1 1 61EB76CD
-P 9850 2400
-F 0 "TP23" H 9908 2518 50  0000 L CNN
-F 1 "TestPoint" H 9908 2427 50  0001 L CNN
-F 2 "" H 10050 2400 50  0001 C CNN
-F 3 "~" H 10050 2400 50  0001 C CNN
-	1    9850 2400
-	1    0    0    1
+P 9950 2300
+F 0 "TP23" V 9950 2500 50  0000 L CNN
+F 1 "TestPoint" H 10008 2327 50  0001 L CNN
+F 2 "" H 10150 2300 50  0001 C CNN
+F 3 "~" H 10150 2300 50  0001 C CNN
+	1    9950 2300
+	0    1    -1   0
 $EndComp
 $Comp
@@
 L Connector:TestPoint TP20
 U 1 1 617B0B48
-P 7950 2450
-F 0 "TP20" H 8008 2568 50  0000 L CNN
-F 1 "TestPoint" H 8008 2477 50  0001 L CNN
-F 2 "" H 8150 2450 50  0001 C CNN
-F 3 "~" H 8150 2450 50  0001 C CNN
-	1    7950 2450
-	-1   0    0    1
+P 8000 2300
+F 0 "TP20" V 8000 2500 50  0000 L CNN
+F 1 "TestPoint" H 8058 2327 50  0001 L CNN
+F 2 "" H 8200 2300 50  0001 C CNN
+F 3 "~" H 8200 2300 50  0001 C CNN
+	1    8000 2300
+	0    -1   -1   0
 $EndComp
 $Comp
@@
 Wire Wire Line
 	8200 2450 8200 2300
-Wire Wire Line
-	7950 2450 7950 2300
 Connection ~ 8200 2300
 Wire Wire Line
 	8200 2300 8300 2300
-Wire Wire Line
-	7950 2300 8200 2300
 Wire Wire Line
 	8200 1900 8200 2000
@@
 Wire Wire Line
 	9300 2300 9600 2300
-Wire Wire Line
-	9850 2400 9850 2300
-Wire Wire Line
-	9600 2300 9850 2300
-Connection ~ 9850 2300
 Wire Wire Line
 	9850 1950 9850 2000
@@
 Text Notes 7950 3150 0    100  ~ 0
 5V Boost Converter\n(Isolation)
-Text Label 7800 2000 0    50   ~ 0
+Text Label 7300 2000 0    50   ~ 0
 +3V3_ni
 Text Label 2350 4400 0    50   ~ 0
@@
 	8200 2000 8300 2000
 Wire Wire Line
-	7750 2000 8200 2000
+	7250 2000 7700 2000
 Wire Wire Line
 	7600 4650 7600 4800
@@
 	2500 1450 3000 1450
 $Comp
-L Device:Jumper_NC_Small JP?
+L Device:Jumper_NC_Small JP3
 U 1 1 619AB4BD
 P 3100 5250
-F 0 "JP?" H 3100 5371 50  0000 C CNN
+F 0 "JP3" H 3100 5371 50  0000 C CNN
 F 1 "Jumper_NC_Small" H 3100 5371 50  0001 C CNN
 F 2 "" H 3100 5250 50  0001 C CNN
@@
 	3000 5250 2700 5250
 $Comp
-L Device:Jumper_NC_Small JP?
+L Device:Jumper_NC_Small JP4
 U 1 1 619AEAC9
 P 4450 2300
-F 0 "JP?" H 4450 2421 50  0000 C CNN
+F 0 "JP4" H 4450 2421 50  0000 C CNN
 F 1 "Jumper_NC_Small" H 4450 2421 50  0001 C CNN
 F 2 "" H 4450 2300 50  0001 C CNN
@@
 Wire Wire Line
 	4350 1550 4800 1550
+$Comp
+L Device:Jumper_NC_Small JP5
+U 1 1 6192FDD4
+P 7800 2000
+F 0 "JP5" H 7800 2121 50  0000 C CNN
+F 1 "Jumper_NC_Small" H 7800 2121 50  0001 C CNN
+F 2 "" H 7800 2000 50  0001 C CNN
+F 3 "~" H 7800 2000 50  0001 C CNN
+	1    7800 2000
+	1    0    0    -1
+$EndComp
+Wire Wire Line
+	7900 2000 8200 2000
+Wire Wire Line
+	8000 2300 8200 2300
+Wire Wire Line
+	9600 2300 9950 2300
 $EndSCHEMATC

Commit message: Updated some footprints and part manufacturers and numbers.
Parts:
- C2, C3, C4, C5, C6: Manufacturer (none) -> Samsung Electro-Mechanics; Part Number (none) -> CL21B104KACNNNC
- D2: footprint (none) -> LED_SMD:LED_0603_1608Metric_Pad1.05x0.95mm_HandSolder; Manufacturer (none) -> Stanley Electric Co; Part Number (none) -> VFHL1116P-4BX3C-TR
- D3: value Blue -> Yellow; footprint (none) -> LED_SMD:LED_0603_1608Metric_Pad1.05x0.95mm_HandSolder; Manufacturer (none) -> VFHY1104P-4C42D-TR; Part Number (none) -> VFHY1104P-4C42D-TR
- JP3, JP4, JP5: footprint (none) -> Jumper:SolderJumper-2_P1.3mm_Bridged_Pad1.0x1.5mm; Manufacturer (none) -> N/A; Part Number (none) -> N/A
- TP10, TP11, TP12, TP13, TP14, TP15, TP16, TP17, TP18, TP19, TP20, TP21, TP22, TP23, TP8, TP9: footprint (none) -> TestPoint:TestPoint_Keystone_5010-5014_Multipurpose; Manufacturer (none) -> N/A; Part Number (none) -> N/A
Changed lines of the file:
@@
 F 2 "Capacitor_SMD:C_0603_1608Metric_Pad1.08x0.95mm_HandSolder" H 4838 1600 50  0001 C CNN
 F 3 "~" H 4800 1750 50  0001 C CNN
+F 4 "Samsung Electro-Mechanics" H 4800 1750 50  0001 C CNN "Manufacturer"
+F 5 "CL21B104KACNNNC" H 4800 1750 50  0001 C CNN "Part Number"
 	1    4800 1750
 	1    0    0    1
@@
 F 2 "Capacitor_SMD:C_0603_1608Metric_Pad1.08x0.95mm_HandSolder" H 3038 1500 50  0001 C CNN
 F 3 "~" H 3000 1650 50  0001 C CNN
+F 4 "Samsung Electro-Mechanics" H 3000 1650 50  0001 C CNN "Manufacturer"
+F 5 "CL21B104KACNNNC" H 3000 1650 50  0001 C CNN "Part Number"
 	1    3000 1650
 	1    0    0    1
@@
 F 0 "TP23" V 9950 2500 50  0000 L CNN
 F 1 "TestPoint" H 10008 2327 50  0001 L CNN
-F 2 "" H 10150 2300 50  0001 C CNN
+F 2 "TestPoint:TestPoint_Keystone_5010-5014_Multipurpose" H 10150 2300 50  0001 C CNN
 F 3 "~" H 10150 2300 50  0001 C CNN
+F 4 "N/A" H 9950 2300 50  0001 C CNN "Manufacturer"
+F 5 "N/A" H 9950 2300 50  0001 C CNN "Part Number"
 	1    9950 2300
 	0    1    -1   0
@@
 F 0 "TP22" H 9908 2068 50  0000 L CNN
 F 1 "TestPoint" H 9908 1977 50  0001 L CNN
-F 2 "" H 10050 1950 50  0001 C CNN
+F 2 "TestPoint:TestPoint_Keystone_5010-5014_Multipurpose" H 10050 1950 50  0001 C CNN
 F 3 "~" H 10050 1950 50  0001 C CNN
+F 4 "N/A" H 9850 1950 50  0001 C CNN "Manufacturer"
+F 5 "N/A" H 9850 1950 50  0001 C CNN "Part Number"
 	1    9850 1950
 	1    0    0    -1
@@
 F 2 "Capacitor_SMD:C_0603_1608Metric_Pad1.08x0.95mm_HandSolder" H 9338 2000 50  0001 C CNN
 F 3 "~" H 9300 2150 50  0001 C CNN
+F 4 "Samsung Electro-Mechanics" H 9300 2150 50  0001 C CNN "Manufacturer"
+F 5 "CL21B104KACNNNC" H 9300 2150 50  0001 C CNN "Part Number"
 	1    9300 2150
 	-1   0    0    1
@@
 F 0 "TP20" V 8000 2500 50  0000 L CNN
 F 1 "TestPoint" H 8058 2327 50  0001 L CNN
-F 2 "" H 8200 2300 50  0001 C CNN
+F 2 "TestPoint:TestPoint_Keystone_5010-5014_Multipurpose" H 8200 2300 50  0001 C CNN
 F 3 "~" H 8200 2300 50  0001 C CNN
+F 4 "N/A" H 8000 2300 50  0001 C CNN "Manufacturer"
+F 5 "N/A" H 8000 2300 50  0001 C CNN "Part Number"
 	1    8000 2300
 	0    -1   -1   0
@@
 F 0 "TP21" H 8258 2018 50  0000 L CNN
 F 1 "TestPoint" H 8258 1927 50  0001 L CNN
-F 2 "" H 8400 1900 50  0001 C CNN
+F 2 "TestPoint:TestPoint_Keystone_5010-5014_Multipurpose" H 8400 1900 50  0001 C CNN
 F 3 "~" H 8400 1900 50  0001 C CNN
+F 4 "N/A" H 8200 1900 50  0001 C CNN "Manufacturer"
+F 5 "N/A" H 8200 1900 50  0001 C CNN "Part Number"
 	1    8200 1900
 	-1   0    0    -1
@@
 F 0 "TP14" H 4650 3100 50  0000 L CNN
 F 1 "TestPoint" H 4350 2900 50  0001 L CNN
-F 2 "" H 4950 2850 50  0001 C CNN
+F 2 "TestPoint:TestPoint_Keystone_5010-5014_Multipurpose" H 4950 2850 50  0001 C CNN
 F 3 "~" H 4950 2850 50  0001 C CNN
+F 4 "N/A" H 4750 2850 50  0001 C CNN "Manufacturer"
+F 5 "N/A" H 4750 2850 50  0001 C CNN "Part Number"
 	1    4750 2850
 	1    0    0    1
@@
 F 0 "TP13" H 2950 3100 50  0000 L CNN
 F 1 "TestPoint" H 3108 2927 50  0001 L CNN
-F 2 "" H 3250 2900 50  0001 C CNN
+F 2 "TestPoint:TestPoint_Keystone_5010-5014_Multipurpose" H 3250 2900 50  0001 C CNN
 F 3 "~" H 3250 2900 50  0001 C CNN
+F 4 "N/A" H 3050 2900 50  0001 C CNN "Manufacturer"
+F 5 "N/A" H 3050 2900 50  0001 C CNN "Part Number"
 	1    3050 2900
 	-1   0    0    1
@@
 F 0 "TP15" H 4850 3300 50  0000 L CNN
 F 1 "TestPoint" H 4550 3100 50  0001 L CNN
-F 2 "" H 5150 3050 50  0001 C CNN
+F 2 "TestPoint:TestPoint_Keystone_5010-5014_Multipurpose" H 5150 3050 50  0001 C CNN
 F 3 "~" H 5150 3050 50  0001 C CNN
+F 4 "N/A" H 4950 3050 50  0001 C CNN "Manufacturer"
+F 5 "N/A" H 4950 3050 50  0001 C CNN "Part Number"
 	1    4950 3050
 	1    0    0    1
@@
 F 0 "TP16" H 5100 3100 50  0000 L CNN
 F 1 "TestPoint" H 4800 2900 50  0001 L CNN
-F 2 "" H 5400 2850 50  0001 C CNN
+F 2 "TestPoint:TestPoint_Keystone_5010-5014_Multipurpose" H 5400 2850 50  0001 C CNN
 F 3 "~" H 5400 2850 50  0001 C CNN
+F 4 "N/A" H 5200 2850 50  0001 C CNN "Manufacturer"
+F 5 "N/A" H 5200 2850 50  0001 C CNN "Part Number"
 	1    5200 2850
 	1    0    0    1
@@
 F 0 "TP18" H 5300 3300 50  0000 L CNN
 F 1 "TestPoint" H 5000 3100 50  0001 L CNN
-F 2 "" H 5600 3050 50  0001 C CNN
+F 2 "TestPoint:TestPoint_Keystone_5010-5014_Multipurpose" H 5600 3050 50  0001 C CNN
 F 3 "~" H 5600 3050 50  0001 C CNN
+F 4 "N/A" H 5400 3050 50  0001 C CNN "Manufacturer"
+F 5 "N/A" H 5400 3050 50  0001 C CNN "Part Number"
 	1    5400 3050
 	1    0    0    1
@@
 F 0 "TP12" H 2750 3050 50  0000 L CNN
 F 1 "TestPoint" H 2908 2877 50  0001 L CNN
-F 2 "" H 3050 2850 50  0001 C CNN
+F 2 "TestPoint:TestPoint_Keystone_5010-5014_Multipurpose" H 3050 2850 50  0001 C CNN
 F 3 "~" H 3050 2850 50  0001 C CNN
+F 4 "N/A" H 2850 2850 50  0001 C CNN "Manufacturer"
+F 5 "N/A" H 2850 2850 50  0001 C CNN "Part Number"
 	1    2850 2850
 	-1   0    0    1
@@
 F 0 "TP10" H 2550 2600 50  0000 L CNN
 F 1 "TestPoint" H 2708 2427 50  0001 L CNN
-F 2 "" H 2850 2400 50  0001 C CNN
+F 2 "TestPoint:TestPoint_Keystone_5010-5014_Multipurpose" H 2850 2400 50  0001 C CNN
 F 3 "~" H 2850 2400 50  0001 C CNN
+F 4 "N/A" H 2650 2400 50  0001 C CNN "Manufacturer"
+F 5 "N/A" H 2650 2400 50  0001 C CNN "Part Number"
 	1    2650 2400
 	1    0    0    -1
@@
 F 0 "TP8" H 2400 2500 50  0000 L CNN
 F 1 "TestPoint" H 2508 2327 50  0001 L CNN
-F 2 "" H 2650 2300 50  0001 C CNN
+F 2 "TestPoint:TestPoint_Keystone_5010-5014_Multipurpose" H 2650 2300 50  0001 C CNN
 F 3 "~" H 2650 2300 50  0001 C CNN
+F 4 "N/A" H 2450 2300 50  0001 C CNN "Manufacturer"
+F 5 "N/A" H 2450 2300 50  0001 C CNN "Part Number"
 	1    2450 2300
 	1    0    0    -1
@@
 F 2 "Capacitor_SMD:C_0603_1608Metric_Pad1.08x0.95mm_HandSolder" H 4688 4550 50  0001 C CNN
 F 3 "~" H 4650 4700 50  0001 C CNN
+F 4 "Samsung Electro-Mechanics" H 4650 4700 50  0001 C CNN "Manufacturer"
+F 5 "CL21B104KACNNNC" H 4650 4700 50  0001 C CNN "Part Number"
 	1    4650 4700
 	1    0    0    1
@@
 F 2 "Capacitor_SMD:C_0603_1608Metric_Pad1.08x0.95mm_HandSolder" H 2888 4450 50  0001 C CNN
 F 3 "~" H 2850 4600 50  0001 C CNN
+F 4 "Samsung Electro-Mechanics" H 2850 4600 50  0001 C CNN "Manufacturer"
+F 5 "CL21B104KACNNNC" H 2850 4600 50  0001 C CNN "Part Number"
 	1    2850 4600
 	-1   0    0    1
@@
 F 0 "TP11" H 2650 5850 50  0000 L CNN
 F 1 "TestPoint" H 2758 5677 50  0001 L CNN
-F 2 "" H 2900 5650 50  0001 C CNN
+F 2 "TestPoint:TestPoint_Keystone_5010-5014_Multipurpose" H 2900 5650 50  0001 C CNN
 F 3 "~" H 2900 5650 50  0001 C CNN
+F 4 "N/A" H 2700 5650 50  0001 C CNN "Manufacturer"
+F 5 "N/A" H 2700 5650 50  0001 C CNN "Part Number"
 	1    2700 5650
 	-1   0    0    1
@@
 F 0 "TP9" H 2450 5750 50  0000 L CNN
 F 1 "TestPoint" H 2558 5577 50  0001 L CNN
-F 2 "" H 2700 5550 50  0001 C CNN
+F 2 "TestPoint:TestPoint_Keystone_5010-5014_Multipurpose" H 2700 5550 50  0001 C CNN
 F 3 "~" H 2700 5550 50  0001 C CNN
+F 4 "N/A" H 2500 5550 50  0001 C CNN "Manufacturer"
+F 5 "N/A" H 2500 5550 50  0001 C CNN "Part Number"
 	1    2500 5550
 	-1   0    0    1
@@
 F 0 "TP19" H 4850 5850 50  0000 L CNN
 F 1 "TestPoint" H 4550 5700 50  0001 L CNN
-F 2 "" H 5150 5650 50  0001 C CNN
+F 2 "TestPoint:TestPoint_Keystone_5010-5014_Multipurpose" H 5150 5650 50  0001 C CNN
 F 3 "~" H 5150 5650 50  0001 C CNN
+F 4 "N/A" H 4950 5650 50  0001 C CNN "Manufacturer"
+F 5 "N/A" H 4950 5650 50  0001 C CNN "Part Number"
 	1    4950 5650
 	1    0    0    1
@@
 F 0 "TP17" H 4550 5800 50  0000 L CNN
 F 1 "TestPoint" H 4250 5650 50  0001 L CNN
-F 2 "" H 4850 5600 50  0001 C CNN
+F 2 "TestPoint:TestPoint_Keystone_5010-5014_Multipurpose" H 4850 5600 50  0001 C CNN
 F 3 "~" H 4850 5600 50  0001 C CNN
+F 4 "N/A" H 4650 5600 50  0001 C CNN "Manufacturer"
+F 5 "N/A" H 4650 5600 50  0001 C CNN "Part Number"
 	1    4650 5600
 	1    0    0    1
@@
 F 0 "D2" H 7700 4800 50  0000 C CNN
 F 1 "Green" H 7500 4800 50  0000 C CNN
-F 2 "" H 7600 4950 50  0001 C CNN
+F 2 "LED_SMD:LED_0603_1608Metric_Pad1.05x0.95mm_HandSolder" H 7600 4950 50  0001 C CNN
 F 3 "~" H 7600 4950 50  0001 C CNN
+F 4 "Stanley Electric Co" H 7600 4950 50  0001 C CNN "Manufacturer"
+F 5 "VFHL1116P-4BX3C-TR" H 7600 4950 50  0001 C CNN "Part Number"
 	1    7600 4950
 	0    -1   -1   0
@@
 AR Path="/61731DC5/618CA26A" Ref="D3"  Part="1"
 F 0 "D3" H 8400 4800 50  0000 C CNN
-F 1 "Blue" H 8200 4800 50  0000 C CNN
-F 2 "" H 8300 4950 50  0001 C CNN
+F 1 "Yellow" H 8200 4800 50  0000 C CNN
+F 2 "LED_SMD:LED_0603_1608Metric_Pad1.05x0.95mm_HandSolder" H 8300 4950 50  0001 C CNN
 F 3 "~" H 8300 4950 50  0001 C CNN
+F 4 "VFHY1104P-4C42D-TR" H 8300 4950 50  0001 C CNN "Manufacturer"
+F 5 "VFHY1104P-4C42D-TR" H 8300 4950 50  0001 C CNN "Part Number"
 	1    8300 4950
 	0    -1   -1   0
@@
 F 0 "JP3" H 3100 5371 50  0000 C CNN
 F 1 "Jumper_NC_Small" H 3100 5371 50  0001 C CNN
-F 2 "" H 3100 5250 50  0001 C CNN
+F 2 "Jumper:SolderJumper-2_P1.3mm_Bridged_Pad1.0x1.5mm" H 3100 5250 50  0001 C CNN
 F 3 "~" H 3100 5250 50  0001 C CNN
+F 4 "N/A" H 3100 5250 50  0001 C CNN "Manufacturer"
+F 5 "N/A" H 3100 5250 50  0001 C CNN "Part Number"
 	1    3100 5250
 	1    0    0    -1
@@
 F 0 "JP4" H 4450 2421 50  0000 C CNN
 F 1 "Jumper_NC_Small" H 4450 2421 50  0001 C CNN
-F 2 "" H 4450 2300 50  0001 C CNN
+F 2 "Jumper:SolderJumper-2_P1.3mm_Bridged_Pad1.0x1.5mm" H 4450 2300 50  0001 C CNN
 F 3 "~" H 4450 2300 50  0001 C CNN
+F 4 "N/A" H 4450 2300 50  0001 C CNN "Manufacturer"
+F 5 "N/A" H 4450 2300 50  0001 C CNN "Part Number"
 	1    4450 2300
 	1    0    0    -1
@@
 F 0 "JP5" H 7800 2121 50  0000 C CNN
 F 1 "Jumper_NC_Small" H 7800 2121 50  0001 C CNN
-F 2 "" H 7800 2000 50  0001 C CNN
+F 2 "Jumper:SolderJumper-2_P1.3mm_Bridged_Pad1.0x1.5mm" H 7800 2000 50  0001 C CNN
 F 3 "~" H 7800 2000 50  0001 C CNN
+F 4 "N/A" H 7800 2000 50  0001 C CNN "Manufacturer"
+F 5 "N/A" H 7800 2000 50  0001 C CNN "Part Number"
 	1    7800 2000
 	1    0    0    -1

Commit message: Finished adding footprints, and started laying out the isolation section.
Parts:
- R18: value 220R -> 1K; Manufacturer (none) -> Stackpole Electronics Inc; Part Number (none) -> RMCF0603FG1K00
- R19: value 330R -> 1K; Manufacturer (none) -> Stackpole Electronics Inc; Part Number (none) -> RMCF0603FG1K00
- U2, U3: footprint (none) -> Package_SO:SOIC-16W_7.5x12.8mm_P1.27mm; Manufacturer (none) -> Analog Devices Inc.; Part Number (none) -> ADUM240E1BRIZ-RL
- U4: footprint MEJ1_SINGLE_SIP_MUR -> VolksEEG:7SIP; Manufacturer (none) -> Murata Power Solutions Inc.; Part Number (none) -> MEJ1S0305SC
Changed lines of the file:
@@
 Text HLabel 9950 2000 2    50   Output ~ 0
 +5V
-Text HLabel 5050 1550 2    50   Input ~ 0
-+3V3
 $Comp
 L VolksEEG:GND_ni #PWR017
@@
 F 0 "U2" H 3775 3137 60  0000 C CNN
 F 1 "ADUM240E1BRIZ-RL" H 3775 3031 60  0000 C CNN
-F 2 "" H 4250 3140 60  0001 C CNN
+F 2 "Package_SO:SOIC-16W_7.5x12.8mm_P1.27mm" H 4250 3140 60  0001 C CNN
 F 3 "" H 3650 2450 60  0000 C CNN
+F 4 "Analog Devices Inc." H 3550 2450 50  0001 C CNN "Manufacturer"
+F 5 "ADUM240E1BRIZ-RL" H 3550 2450 50  0001 C CNN "Part Number"
 	1    3550 2450
 	1    0    0    -1
@@
 Wire Wire Line
 	2450 2450 3350 2450
-Wire Wire Line
-	5000 2300 4550 2300
 $Comp
 L VolksEEG:GND_ni #PWR07
@@
 F 0 "U3" H 4275 6087 60  0000 C CNN
 F 1 "ADUM240E1BRIZ-RL" H 4275 5981 60  0000 C CNN
-F 2 "" H 4750 6090 60  0001 C CNN
+F 2 "Package_SO:SOIC-16W_7.5x12.8mm_P1.27mm" H 4750 6090 60  0001 C CNN
 F 3 "" H 4150 5400 60  0000 C CNN
+F 4 "Analog Devices Inc." H 4050 5400 50  0001 C CNN "Manufacturer"
+F 5 "ADUM240E1BRIZ-RL" H 4050 5400 50  0001 C CNN "Part Number"
 	1    4050 5400
 	-1   0    0    -1
@@
 F 0 "U4" H 8750 2587 60  0000 C CNN
 F 1 "MEJ1S0305SC" H 8750 2481 60  0000 C CNN
-F 2 "MEJ1_SINGLE_SIP_MUR" H 8750 2440 60  0001 C CNN
+F 2 "VolksEEG:7SIP" H 8750 2440 60  0001 C CNN
 F 3 "" H 8750 1950 60  0000 C CNN
+F 4 "Murata Power Solutions Inc." H 8750 2150 50  0001 C CNN "Manufacturer"
+F 5 "MEJ1S0305SC" H 8750 2150 50  0001 C CNN "Part Number"
 	1    8750 2150
 	1    0    0    -1
@@
 AR Path="/61731DC5/618CCE2C" Ref="R19"  Part="1"
 F 0 "R19" V 8093 5450 50  0000 C CNN
-F 1 "330R" V 8184 5450 50  0000 C CNN
+F 1 "1K" V 8184 5450 50  0000 C CNN
 F 2 "Resistor_SMD:R_0603_1608Metric_Pad0.98x0.95mm_HandSolder" V 8230 5450 50  0001 C CNN
-F 3 "~" H 8300 5450 50  0001 C CNN
+F 3 "https://www.seielect.com/catalog/sei-rmcf_rmcp.pdf" H 8300 5450 50  0001 C CNN
+F 4 "Stackpole Electronics Inc" H 8300 5450 50  0001 C CNN "Manufacturer"
+F 5 "RMCF0603FG1K00" H 8300 5450 50  0001 C CNN "Part Number"
 	1    8300 5450
 	-1   0    0    1
@@
 AR Path="/61731DC5/618CA270" Ref="R18"  Part="1"
 F 0 "R18" V 7393 5450 50  0000 C CNN
-F 1 "220R" V 7484 5450 50  0000 C CNN
+F 1 "1K" V 7484 5450 50  0000 C CNN
 F 2 "Resistor_SMD:R_0603_1608Metric_Pad0.98x0.95mm_HandSolder" V 7530 5450 50  0001 C CNN
-F 3 "~" H 7600 5450 50  0001 C CNN
+F 3 "https://www.seielect.com/catalog/sei-rmcf_rmcp.pdf" H 7600 5450 50  0001 C CNN
+F 4 "Stackpole Electronics Inc" H 7600 5450 50  0001 C CNN "Manufacturer"
+F 5 "RMCF0603FG1K00" H 7600 5450 50  0001 C CNN "Part Number"
 	1    7600 5450
 	-1   0    0    1
@@
 	0    -1   -1   0
 $EndComp
-Text Label 5000 2300 2    50   ~ 0
-+3V3_ni
 Text Label 5150 4500 2    50   ~ 0
 +3V3
@@
 Wire Wire Line
 	7600 4650 7350 4650
-Text Label 2700 5250 0    50   ~ 0
-+3V3
 Connection ~ 4650 5500
 Wire Wire Line
@@
 Wire Wire Line
 	2850 4400 3250 4400
-Wire Wire Line
-	2350 4400 2850 4400
 Connection ~ 3000 1450
 Wire Wire Line
@@
 	1    0    0    -1
 $EndComp
-Wire Wire Line
-	3000 5250 2700 5250
 $Comp
 L Device:Jumper_NC_Small JP4
@@
 Connection ~ 4800 1550
 Wire Wire Line
-	4800 1550 5050 1550
-Wire Wire Line
 	4350 1550 4800 1550
 $Comp
@@
 Wire Wire Line
 	9600 2300 9950 2300
+Wire Wire Line
+	5000 2300 4550 2300
+Wire Wire Line
+	4800 1550 5050 1550
+Text HLabel 5050 1550 2    50   Input ~ 0
++3V3
+Text Label 5000 2300 2    50   ~ 0
++3V3
+Wire Wire Line
+	2350 4400 2850 4400
+Wire Wire Line
+	3000 5250 2700 5250
+Text Label 2700 5250 0    50   ~ 0
++3V3_ni
 $EndSCHEMATC

Commit message: Layout of the NRF52840 section of the PCB.
Changed lines of the file:
@@
 Text Label 2700 5250 0    50   ~ 0
 +3V3_ni
+Wire Notes Line
+	4750 2150 4750 2400
+Wire Notes Line
+	4750 2400 5150 2400
+Wire Notes Line
+	5150 2400 5150 2150
+Wire Notes Line
+	5150 2150 4750 2150
+Wire Notes Line
+	2650 5100 2650 5350
+Wire Notes Line
+	2650 5350 3050 5350
+Wire Notes Line
+	3050 5350 3050 5100
+Wire Notes Line
+	3050 5100 2650 5100
 $EndSCHEMATC
