File: hardware/KiCAD/VolksEEG/Power.sch (KiCad schematic (older format))
At the start: 44 parts, among them U5 LP3990MF-3.3, U6 ADP7182ACPZ-2.5-R7, U7 TPS78425Q, U8 LM2660MX

Commit message: Updated some footprints and part manufacturers and numbers.
Parts:
- C16, C17, C18, C19, C20, C21: Manufacturer (none) -> Samsung Electro-Mechanics; Part Number (none) -> CL21B225KAFNFNE
- C22, C23, C24, C25, C26, C28, C30, C39, C41: Manufacturer (none) -> Samsung Electro-Mechanics; Part Number (none) -> CL21B106KPQNNNE
- C27, C31, C32, C35, C38: footprint (none) -> Capacitor_SMD:C_0603_1608Metric_Pad1.08x0.95mm_HandSolder; Manufacturer (none) -> Samsung Electro-Mechanics; Part Number (none) -> CL21B104KACNNNC
- C29, C37: Manufacturer (none) -> Samsung Electro-Mechanics; Part Number (none) -> CL21B105KAFNNNE
- C33, C34, C36, C40: footprint (none) -> Capacitor_SMD:C_0603_1608Metric_Pad1.08x0.95mm_HandSolder; Manufacturer (none) -> Samsung Electro-Mechanics; Part Number (none) -> CL21B105KAFNNNE
- JP1, JP2: Manufacturer (none) -> N/A; Part Number (none) -> N/A
- L1, L2, L3, L4: footprint (none) -> Inductor_SMD:L_0805_2012Metric_Pad1.15x1.40mm_HandSolder; Manufacturer (none) -> TDK Corporation; Part Number (none) -> MLZ2012A3R3WTD25
- TP24, TP26: footprint TestPoint:TestPoint_Keystone_5010-5014_Multipurpose -> TestPoint:TestPoint_Bridge_Pitch7.62mm_Drill1.3mm; Manufacturer (none) -> N/A; Part Number (none) -> N/A
- TP25, TP27, TP28, TP29, TP30: footprint (none) -> TestPoint:TestPoint_Keystone_5010-5014_Multipurpose; Manufacturer (none) -> N/A; Part Number (none) -> N/A

Commit message: Finished adding footprints, and started laying out the isolation section.
Parts:
- R31: Manufacturer (none) -> Rohm Semiconductor; Part Number (none) -> TRR03EZPJ000
- U5: Manufacturer (none) -> Texas Instruments; Part Number (none) -> LP3990MF-3.3
- U6: footprint (none) -> Package_CSP:LFCSP-8-1EP_3x3mm_P0.5mm_EP1.45x1.74mm; Manufacturer (none) -> Analog Devices Inc.; Part Number (none) -> ADP7182ACPZN-2.5R7
- U7: Manufacturer (none) -> Texas Instruments; Part Number (none) -> TPS78425QDBVRQ1
- U8: Manufacturer (none) -> Texas Instruments; Part Number (none) -> LM2660MX
Changed lines of the file:
@@
 F 4 "https://www.digikey.com/en/products/detail/texas-instruments/LM2660MX-NOPB/366876?s=N4IgTCBcDaIDIFkwDZkAYEA0D0A5A8gAoBCABCALoC%2BQA" H 8000 1650 50  0001 C CNN "Supplier 1 Link"
 F 5 "https://eu.mouser.com/ProductDetail/Texas-Instruments/LM2660MX-NOPB?qs=%2Fha2pyFadugHGOygNHaYnDjgJHODW6F6O01kwvJjsKBnt2qN9JbSfA%3D%3D" H 8000 1650 50  0001 C CNN "Supplier 2 Link"
+F 6 "Texas Instruments" H 8000 1650 50  0001 C CNN "Manufacturer"
+F 7 "LM2660MX" H 8000 1650 50  0001 C CNN "Part Number"
 	1    8000 1650
 	1    0    0    -1
@@
 F 2 "Resistor_SMD:R_0603_1608Metric_Pad0.98x0.95mm_HandSolder" V 4230 1850 50  0001 C CNN
 F 3 "~" H 4300 1850 50  0001 C CNN
+F 4 "Rohm Semiconductor" H 4300 1850 50  0001 C CNN "Manufacturer"
+F 5 "TRR03EZPJ000" H 4300 1850 50  0001 C CNN "Part Number"
 	1    4300 1850
 	0    1    1    0
@@
 F 0 "U6" H 3050 5800 60  0000 C CNN
 F 1 "ADP7182ACPZ-2.5-R7" H 3050 5700 60  0000 C CNN
-F 2 "" H 3850 5690 60  0001 C CNN
+F 2 "Package_CSP:LFCSP-8-1EP_3x3mm_P0.5mm_EP1.45x1.74mm" H 3850 5690 60  0001 C CNN
 F 3 "" H 3050 5350 60  0000 C CNN
+F 4 "Analog Devices Inc." H 3050 5350 50  0001 C CNN "Manufacturer"
+F 5 "ADP7182ACPZN-2.5R7" H 3050 5350 50  0001 C CNN "Part Number"
 	1    3050 5350
 	1    0    0    -1
@@
 F 4 "https://www.digikey.com/en/products/detail/texas-instruments/LP3990MF-3-3-NOPB/953453?s=N4IgTCBcDaIDIAUDMBOFAGAsgMQLRIDokB6AOQHkEAhAAhAF0BfIA" H 3150 650 50  0001 C CNN "Supplier 1 Link"
 F 5 "https://eu.mouser.com/ProductDetail/Texas-Instruments/LP3990MF-33-NOPB?qs=1FNqv8aZn1ScRIqY9rNFxg%3D%3D" H 3300 1000 50  0001 C CNN "Supplier 2 Link"
+F 6 "Texas Instruments" H 2800 1500 50  0001 C CNN "Manufacturer"
+F 7 "LP3990MF-3.3" H 2800 1500 50  0001 C CNN "Part Number"
 	1    2800 1500
 	1    0    0    -1
@@
 F 4 "https://www.digikey.com/en/products/detail/texas-instruments/TPS78425QDBVRQ1/13563001" H 0   0   50  0001 C CNN "Supplier 1 Link"
 F 5 "https://eu.mouser.com/ProductDetail/Texas-Instruments/TPS78425QDBVRQ1?qs=81r%252BiQLm7BRHMcAKEdEeyg%3D%3D" H 0   0   50  0001 C CNN "Supplier 2 Link"
+F 6 "Texas Instruments" H 3100 3700 50  0001 C CNN "Manufacturer"
+F 7 "TPS78425QDBVRQ1" H 3100 3700 50  0001 C CNN "Part Number"
 	1    3100 3700
 	1    0    0    -1

Commit message: Further PCB Layout.
Parts:
- U6: footprint Package_CSP:LFCSP-8-1EP_3x3mm_P0.5mm_EP1.45x1.74mm -> Package_TO_SOT_SMD:TSOT-23-5
Changed lines of the file:
@@
 F 0 "U6" H 3050 5800 60  0000 C CNN
 F 1 "ADP7182ACPZ-2.5-R7" H 3050 5700 60  0000 C CNN
-F 2 "Package_CSP:LFCSP-8-1EP_3x3mm_P0.5mm_EP1.45x1.74mm" H 3850 5690 60  0001 C CNN
+F 2 "Package_TO_SOT_SMD:TSOT-23-5" H 3850 5690 60  0001 C CNN
 F 3 "" H 3050 5350 60  0000 C CNN
 F 4 "Analog Devices Inc." H 3050 5350 50  0001 C CNN "Manufacturer"
