File: hardware/KiCAD/VolksEEG/VolksEEG.kicad_pcb (KiCad board)
At the start: 4 copper layers, 70 x 75 mm, 48 parts, among them J1 Conn_02x13_Odd_Even, U1 ADS1299IPAG, U2 nRF52840-Feather-Sense, U3 LP3990MF-3.3, U4 LM2660MX, U5 TPS78425Q, U6 TPS72325Q

Commit message: Update
Parts:
- added J2: 693061010911, VolksEEG:693061010911, F.Cu at (68.6, 56.1)
- added R17: R, Resistor_SMD:R_0603_1608Metric_Pad0.98x0.95mm_HandSolder, F.Cu at (166.6, 48.1)
- added R18: R, Resistor_SMD:R_0603_1608Metric_Pad0.98x0.95mm_HandSolder, F.Cu at (166.6, 50.6)
- added U7: ISO7761DW, Package_SO:SOIC-16W_7.5x10.3mm_P1.27mm, F.Cu at (72.4, 102.6)
- added U8: UCC12050DVER, VolksEEG:SOIC127P1030X265-16N, F.Cu at (102.1, 109.7)
- moved C10 57.0 mm to (81.5, 133.8)
- moved C11 57.0 mm to (83.1, 133.8)
- moved C12 57.0 mm to (78.5, 133.8)
- moved C13 57.0 mm to (80.0, 133.8)
- moved C14 57.0 mm to (75.4, 133.8)
- moved C15 57.0 mm to (77.0, 133.8)
- moved C16 57.0 mm to (72.4, 133.8)
- moved C17 57.0 mm to (73.9, 133.8)
- moved C18 57.0 mm to (66.3, 133.8)
- moved C19 57.0 mm to (67.8, 133.8)
- moved C20 57.0 mm to (69.3, 133.8)
- moved C21 57.0 mm to (70.9, 133.8)
- moved C22 57.0 mm to (63.2, 133.8)
- moved C23 57.0 mm to (64.8, 133.8)
- moved C24 57.0 mm to (60.2, 133.8)
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Connections:
- U2 pad 11: /ADS1299/SCK -> /nRF52840/SCK
- U2 pad 12: /ADS1299/MOSI -> /nRF52840/MOSI
- U2 pad 13: /ADS1299/MISO -> /nRF52840/MISO
- U2 pad 19: /ADS1299/nCS -> /nRF52840/nCS0
- U2 pad 20: /ADS1299/ADS-nRST -> /nRF52840/nCS1
- U2 pad 21: Net-(U2-Pad21) -> /nRF52840/ADS-nRST
Other:
- board size 70 x 75 mm -> 100 x 100 mm

Commit message: Finished adding footprints, and started laying out the isolation section.
Parts:
- removed R13: R, Resistor_SMD:R_0603_1608Metric_Pad0.98x0.95mm_HandSolder
- added C26: 10u, Capacitor_SMD:C_0603_1608Metric_Pad1.08x0.95mm_HandSolder, F.Cu at (384.1, 122.2)
- added C27: 100n, Capacitor_SMD:C_0603_1608Metric_Pad1.08x0.95mm_HandSolder, F.Cu at (375.0, 130.2)
- added C28: 10u, Capacitor_SMD:C_0603_1608Metric_Pad1.08x0.95mm_HandSolder, F.Cu at (375.0, 127.7)
- added C29: 1u, Capacitor_SMD:C_0603_1608Metric_Pad1.08x0.95mm_HandSolder, F.Cu at (384.3, 117.2)
- added C30: 10u, Capacitor_SMD:C_0603_1608Metric_Pad1.08x0.95mm_HandSolder, F.Cu at (379.7, 122.2)
- added C31: 100n, Capacitor_SMD:C_0603_1608Metric_Pad1.08x0.95mm_HandSolder, F.Cu at (370.6, 129.8)
- added C32: 100n, Capacitor_SMD:C_0603_1608Metric_Pad1.08x0.95mm_HandSolder, F.Cu at (371.0, 122.2)
- added C33: 1u, Capacitor_SMD:C_0603_1608Metric_Pad1.08x0.95mm_HandSolder, F.Cu at (370.6, 127.3)
- added C34: 1u, Capacitor_SMD:C_0603_1608Metric_Pad1.08x0.95mm_HandSolder, F.Cu at (375.4, 122.7)
- added C35: 100n, Capacitor_SMD:C_0603_1608Metric_Pad1.08x0.95mm_HandSolder, F.Cu at (380.0, 119.7)
- added C36: 1u, Capacitor_SMD:C_0603_1608Metric_Pad1.08x0.95mm_HandSolder, F.Cu at (375.4, 120.1)
- added C37: 1u, Capacitor_SMD:C_0603_1608Metric_Pad1.08x0.95mm_HandSolder, F.Cu at (363.7, 133.7)
- added C38: 100n, Capacitor_SMD:C_0603_1608Metric_Pad1.08x0.95mm_HandSolder, F.Cu at (365.6, 130.1)
- added C39: 10u, Capacitor_SMD:C_0603_1608Metric_Pad1.08x0.95mm_HandSolder, F.Cu at (371.0, 124.8)
- added C40: 1u, Capacitor_SMD:C_0603_1608Metric_Pad1.08x0.95mm_HandSolder, F.Cu at (380.0, 117.2)
- added C41: 10u, Capacitor_SMD:C_0603_1608Metric_Pad1.08x0.95mm_HandSolder, F.Cu at (368.1, 132.7)
- added C42: 10u, Capacitor_SMD:C_0603_1608Metric_Pad1.08x0.95mm_HandSolder, F.Cu at (418.3, 124.7)
- added C43: 100n, Capacitor_SMD:C_0603_1608Metric_Pad1.08x0.95mm_HandSolder, F.Cu at (418.3, 122.2)
- added C44: 100n, Capacitor_SMD:C_0603_1608Metric_Pad1.08x0.95mm_HandSolder, F.Cu at (407.0, 131.9)
- added C45: 1u, Capacitor_SMD:C_0603_1608Metric_Pad1.08x0.95mm_HandSolder, F.Cu at (413.9, 124.7)
- added C46: 1u, Capacitor_SMD:C_0603_1608Metric_Pad1.08x0.95mm_HandSolder, F.Cu at (406.7, 129.4)
- added C47: 1u, Capacitor_SMD:C_0603_1608Metric_Pad1.08x0.95mm_HandSolder, F.Cu at (398.3, 131.6)
- added C48: 100n, Capacitor_SMD:C_0603_1608Metric_Pad1.08x0.95mm_HandSolder, F.Cu at (413.9, 122.2)
- added C49: 1u, Capacitor_SMD:C_0603_1608Metric_Pad1.08x0.95mm_HandSolder, F.Cu at (413.9, 117.2)
- added C50: 100n, Capacitor_SMD:C_0603_1608Metric_Pad1.08x0.95mm_HandSolder, F.Cu at (402.6, 131.9)
- added C51: 100n, Capacitor_SMD:C_0603_1608Metric_Pad1.08x0.95mm_HandSolder, F.Cu at (418.3, 117.2)
- added C52: 1u, Capacitor_SMD:C_0603_1608Metric_Pad1.08x0.95mm_HandSolder, F.Cu at (413.9, 119.7)
- added C53: 100n, Capacitor_SMD:C_0603_1608Metric_Pad1.08x0.95mm_HandSolder, F.Cu at (411.1, 129.4)
- added C54: 1u, Capacitor_SMD:C_0603_1608Metric_Pad1.08x0.95mm_HandSolder, F.Cu at (418.3, 119.7)
- added C55: 100u, Capacitor_SMD:C_1210_3225Metric_Pad1.33x2.70mm_HandSolder, F.Cu at (393.1, 132.5)
- added D1: Red, LED_SMD:LED_0603_1608Metric_Pad1.05x0.95mm_HandSolder, F.Cu at (349.0, 95.6)
- added D2: Green, LED_SMD:LED_0603_1608Metric_Pad1.05x0.95mm_HandSolder, F.Cu at (85.0, 169.7)
- added D3: Yellow, LED_SMD:LED_0603_1608Metric_Pad1.05x0.95mm_HandSolder, F.Cu at (80.6, 169.7)
- added J3: 693061010911, VolksEEG:693061010911, F.Cu at (354.3, 53.3)
- added J4: Conn_01x10, Connector_PinHeader_2.54mm:PinHeader_1x10_P2.54mm_Vertical, F.Cu at (437.6, 67.2)
- added J5: Conn_02x04_Counter_Clockwise, Connector_PinHeader_2.54mm:PinHeader_2x04_P2.54mm_Vertical, F.Cu at (406.9, 118.3)
- added JP1: Jumper_NO_Small, Jumper:SolderJumper-2_P1.3mm_Open_Pad1.0x1.5mm, F.Cu at (363.7, 136.8)
- added JP2: Jumper_NC_Small, Jumper:SolderJumper-2_P1.3mm_Bridged_Pad1.0x1.5mm, F.Cu at (366.3, 127.1)
- added JP3: Jumper_NC_Small, Jumper:SolderJumper-2_P1.3mm_Bridged_Pad1.0x1.5mm, F.Cu at (37.8, 149.1)
- added JP4: Jumper_NC_Small, Jumper:SolderJumper-2_P1.3mm_Bridged_Pad1.0x1.5mm, F.Cu at (26.9, 132.8)
- added JP5: Jumper_NC_Small, Jumper:SolderJumper-2_P1.3mm_Bridged_Pad1.0x1.5mm, F.Cu at (57.5, 151.9)
- added L1: 3.3u, Inductor_SMD:L_0805_2012Metric_Pad1.15x1.40mm_HandSolder, F.Cu at (366.5, 123.9)
- added L2: 3.3u, Inductor_SMD:L_0805_2012Metric_Pad1.15x1.40mm_HandSolder, F.Cu at (349.1, 136.4)
- added L3: 3.3u, Inductor_SMD:L_0805_2012Metric_Pad1.15x1.40mm_HandSolder, F.Cu at (375.4, 117.4)
- added L4: 3.3u, Inductor_SMD:L_0805_2012Metric_Pad1.15x1.40mm_HandSolder, F.Cu at (353.9, 136.4)
- added R19: 1K, Resistor_SMD:R_0603_1608Metric_Pad0.98x0.95mm_HandSolder, F.Cu at (75.3, 176.5)
- added R20: 1M, Resistor_SMD:R_0603_1608Metric_Pad0.98x0.95mm_HandSolder, F.Cu at (460.8, 69.1)
- added R21: 4.99k, Resistor_SMD:R_0603_1608Metric_Pad0.98x0.95mm_HandSolder, F.Cu at (450.8, 77.2)
- added R22: 4.99k, Resistor_SMD:R_0603_1608Metric_Pad0.98x0.95mm_HandSolder, F.Cu at (446.4, 77.2)
- added R23: 4.99k, Resistor_SMD:R_0603_1608Metric_Pad0.98x0.95mm_HandSolder, F.Cu at (442.1, 77.2)
- added R24: 4.99k, Resistor_SMD:R_0603_1608Metric_Pad0.98x0.95mm_HandSolder, F.Cu at (455.1, 74.2)
- added R25: 4.99k, Resistor_SMD:R_0603_1608Metric_Pad0.98x0.95mm_HandSolder, F.Cu at (450.8, 74.7)
- added R26: 4.99k, Resistor_SMD:R_0603_1608Metric_Pad0.98x0.95mm_HandSolder, F.Cu at (446.4, 74.7)
- added R27: 4.99k, Resistor_SMD:R_0603_1608Metric_Pad0.98x0.95mm_HandSolder, F.Cu at (456.5, 69.1)
- added R28: 4.99k, Resistor_SMD:R_0603_1608Metric_Pad0.98x0.95mm_HandSolder, F.Cu at (450.8, 72.1)
- added R29: 4.99k, Resistor_SMD:R_0603_1608Metric_Pad0.98x0.95mm_HandSolder, F.Cu at (456.5, 71.6)
- added R30: 4.99k, Resistor_SMD:R_0603_1608Metric_Pad0.98x0.95mm_HandSolder, F.Cu at (442.1, 74.2)
- added R31: 0R, Resistor_SMD:R_0603_1608Metric_Pad0.98x0.95mm_HandSolder, F.Cu at (379.7, 124.7)
- added R32: 10K, Resistor_SMD:R_0603_1608Metric_Pad0.98x0.95mm_HandSolder, F.Cu at (420.0, 129.7)
- added R33: 10K, Resistor_SMD:R_0603_1608Metric_Pad0.98x0.95mm_HandSolder, F.Cu at (415.7, 132.2)
- added R34: 10K, Resistor_SMD:R_0603_1608Metric_Pad0.98x0.95mm_HandSolder, F.Cu at (415.7, 129.7)
- added R35: 10K, Resistor_SMD:R_0603_1608Metric_Pad0.98x0.95mm_HandSolder, F.Cu at (419.8, 127.2)
- added R36: 10K, Resistor_SMD:R_0603_1608Metric_Pad0.98x0.95mm_HandSolder, F.Cu at (411.3, 131.9)
- added R37: 10K, Resistor_SMD:R_0603_1608Metric_Pad0.98x0.95mm_HandSolder, F.Cu at (415.4, 127.2)
- added TP1: TestPoint, TestPoint:TestPoint_Keystone_5010-5014_Multipurpose, F.Cu at (374.1, 90.2)
- added TP10: TestPoint, TestPoint:TestPoint_Keystone_5010-5014_Multipurpose, F.Cu at (24.4, 166.1)
- added TP11: TestPoint, TestPoint:TestPoint_Keystone_5010-5014_Multipurpose, F.Cu at (40.9, 157.2)
- added TP12: TestPoint, TestPoint:TestPoint_Keystone_5010-5014_Multipurpose, F.Cu at (24.4, 155.7)
- added TP13: TestPoint, TestPoint:TestPoint_Keystone_5010-5014_Multipurpose, F.Cu at (29.0, 159.8)
- added TP14: TestPoint, TestPoint:TestPoint_Keystone_5010-5014_Multipurpose, F.Cu at (-4.32, 109.5)
- added TP15: TestPoint, TestPoint:TestPoint_Keystone_5010-5014_Multipurpose, F.Cu at (-7.37, 118.9)
- added TP16: TestPoint, TestPoint:TestPoint_Keystone_5010-5014_Multipurpose, F.Cu at (-3.56, 124.0)
- added TP17: TestPoint, TestPoint:TestPoint_Keystone_5010-5014_Multipurpose, F.Cu at (41.9, 121.9)
- added TP18: TestPoint, TestPoint:TestPoint_Keystone_5010-5014_Multipurpose, F.Cu at (-2.29, 115.1)
- added TP19: TestPoint, TestPoint:TestPoint_Keystone_5010-5014_Multipurpose, F.Cu at (39.9, 129.5)
- added TP2: TestPoint, TestPoint:TestPoint_Keystone_5010-5014_Multipurpose, F.Cu at (369.1, 90.2)
- added TP20: TestPoint, TestPoint:TestPoint_Keystone_5010-5014_Multipurpose, F.Cu at (69.8, 144.8)
- added TP21: TestPoint, TestPoint:TestPoint_Keystone_5010-5014_Multipurpose, F.Cu at (69.8, 152.4)
- added TP22: TestPoint, TestPoint:TestPoint_Keystone_5010-5014_Multipurpose, F.Cu at (53.3, 124.5)
- added TP23: TestPoint, TestPoint:TestPoint_Keystone_5010-5014_Multipurpose, F.Cu at (69.8, 137.2)
- added TP24: TestPoint, TestPoint:TestPoint_Bridge_Pitch7.62mm_Drill1.3mm, F.Cu at (349.1, 122.9)
- added TP25: TestPoint, TestPoint:TestPoint_Keystone_5010-5014_Multipurpose, F.Cu at (361.6, 124.9)
- added TP26: TestPoint, TestPoint:TestPoint_Bridge_Pitch7.62mm_Drill1.3mm, F.Cu at (349.1, 118.3)
- added TP27: TestPoint, TestPoint:TestPoint_Keystone_5010-5014_Multipurpose, F.Cu at (370.5, 118.5)
- added TP28: TestPoint, TestPoint:TestPoint_Keystone_5010-5014_Multipurpose, F.Cu at (354.3, 132.4)
- added TP29: TestPoint, TestPoint:TestPoint_Keystone_5010-5014_Multipurpose, F.Cu at (360.9, 130.0)
- added TP3: TestPoint, TestPoint:TestPoint_Keystone_5010-5014_Multipurpose, F.Cu at (353.9, 104.3)
- added TP30: TestPoint, TestPoint:TestPoint_Keystone_5010-5014_Multipurpose, F.Cu at (349.3, 132.4)
- added TP31: TestPoint, TestPoint:TestPoint_Bridge_Pitch7.62mm_Drill1.3mm, F.Cu at (349.1, 99.5)
- added TP4: TestPoint, TestPoint:TestPoint_Keystone_5010-5014_Multipurpose, F.Cu at (359.0, 104.3)
- added TP5: TestPoint, TestPoint:TestPoint_Keystone_5010-5014_Multipurpose, F.Cu at (364.0, 102.5)
- added TP6: TestPoint, TestPoint:TestPoint_Keystone_5010-5014_Multipurpose, F.Cu at (384.2, 90.2)
- added TP7: TestPoint, TestPoint:TestPoint_Keystone_5010-5014_Multipurpose, F.Cu at (379.2, 90.2)
- added TP8: TestPoint, TestPoint:TestPoint_Keystone_5010-5014_Multipurpose, F.Cu at (20.3, 160.3)
- added TP9: TestPoint, TestPoint:TestPoint_Keystone_5010-5014_Multipurpose, F.Cu at (45.7, 158.8)
- added U9: ADS1299IPAG, Package_QFP:LQFP-64_10x10mm_P0.5mm, F.Cu at (397.3, 123.2)
- C1, C3, C5, C6: value 1u -> 100n
- C10: value C -> 1.5n; moved to F.Cu
- C11, C12, C13, C14, C15: value C -> 33n; footprint Capacitor_SMD:C_0603_1608Metric_Pad1.08x0.95mm_HandSolder -> Capacitor_SMD:C_0805_2012Metric_Pad1.18x1.45mm_HandSolder; moved to F.Cu
- C16, C17, C18, C19, C20, C21: value C -> 2.2u; moved to F.Cu
- C2, C4: value 10u -> 100n
- C22, C23, C24, C25: value C -> 10u; moved to F.Cu
- C7: value C -> 33n; footprint Capacitor_SMD:C_0603_1608Metric_Pad1.08x0.95mm_HandSolder -> Capacitor_SMD:C_0805_2012Metric_Pad1.18x1.45mm_HandSolder
- C8, C9: value 2.2u -> 33n; footprint Capacitor_SMD:C_0603_1608Metric_Pad1.08x0.95mm_HandSolder -> Capacitor_SMD:C_0805_2012Metric_Pad1.18x1.45mm_HandSolder
- J1: value Conn_02x13_Odd_Even -> Conn_01x03; footprint Connector_PinHeader_2.54mm:PinHeader_2x13_P2.54mm_Vertical -> Connector_PinHeader_2.54mm:PinHeader_1x03_P2.54mm_Vertical
- J2: value 693061010911 -> QWIIC; footprint VolksEEG:693061010911 -> Connector_PinHeader_2.54mm:PinHeader_1x04_P2.54mm_Vertical
- R1, R14, R15, R16, R2, R4, R5, R6, R7: value R -> 0R
- R10, R11, R12, R8, R9: value R -> 4K7
- R17: value R -> 2R2; footprint Resistor_SMD:R_0603_1608Metric_Pad0.98x0.95mm_HandSolder -> VolksEEG:high_power_chip_resistor
- R18, R3: value R -> 1K
- U1: value ADS1299IPAG -> nRF52840-Feather-Sense-Board; footprint VolksEEG:QFP50P1200X1200X120-64N -> VolksEEG:nRF52840_Feather_Sense
- U2: value nRF52840-Feather-Sense -> ADUM240E1BRIZ-RL; footprint VolksEEG:nRF52840_Feather_Sense -> Package_SO:SOIC-16W_7.5x12.8mm_P1.27mm
- U3: value LP3990MF-3.3 -> ADUM240E1BRIZ-RL; footprint VolksEEG:SOT95P280X145-5N -> Package_SO:SOIC-16W_7.5x12.8mm_P1.27mm
- U4: value LM2660MX -> MEJ1S0305SC; footprint VolksEEG:SOIC127P599X175-8N -> VolksEEG:7SIP
- U5: value TPS78425Q -> LP3990MF-3.3; footprint VolksEEG:SOT95P280X145-5N -> Package_TO_SOT_SMD:SOT-23-5_HandSoldering
- U6: value TPS72325Q -> ADP7182ACPZ-2.5-R7; footprint VolksEEG:SOT95P280X145-5N -> Package_CSP:LFCSP-8-1EP_3x3mm_P0.5mm_EP1.45x1.74mm
- U7: value ISO7761DW -> TPS78425Q; footprint Package_SO:SOIC-16W_7.5x10.3mm_P1.27mm -> Package_TO_SOT_SMD:SOT-23-5_HandSoldering
- U8: value UCC12050DVER -> LM2660MX; footprint VolksEEG:SOIC127P1030X265-16N -> VolksEEG:SOIC127P599X175-8N
- moved C12 384.2 mm to (456.7, 66.4), turned to 0 degrees
- moved C13 377.9 mm to (451.9, 66.4), turned to 0 degrees
- moved C14 377.7 mm to (447.1, 66.4), turned to 0 degrees
- moved C11 374.4 mm to (451.9, 69.4), turned to 0 degrees
- moved C15 371.5 mm to (442.3, 66.4), turned to 0 degrees
- moved C10 370.0 mm to (446.4, 72.1), turned to 0 degrees
- moved C7 340.7 mm to (461.5, 66.4)
- moved R16 330.8 mm to (388.9, 89.0), turned to 0 degrees
- moved R9 329.9 mm to (393.3, 94.0), turned to 0 degrees
- moved R11 327.2 mm to (393.3, 91.5), turned to 0 degrees
- moved C9 324.8 mm to (447.1, 69.4), turned to 0 degrees
- moved R10 324.1 mm to (388.9, 94.0), turned to 0 degrees
- moved R12 321.4 mm to (388.9, 91.5), turned to 0 degrees
- moved C8 319.8 mm to (442.3, 69.4), turned to 0 degrees
- moved R3 318.6 mm to (393.3, 89.0), turned to 0 degrees
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Connections:
- C1 pad 1: VDC -> GND
- C1 pad 2: GND -> Net-(C1-Pad2)
- C10 pad 1: /ADS1299/AIN1N -> /ADS1299/BIAS_OUT
- C10 pad 2: GND -> /ADS1299/BIAS_INV
- C11 pad 1: GND -> /ADS1299/AIN5
- C11 pad 2: /ADS1299/AIN1P -> /ADS1299/REF
- C12 pad 1: /ADS1299/AIN2N -> /ADS1299/AIN4
- C12 pad 2: GND -> /ADS1299/REF
- C13 pad 1: GND -> /ADS1299/AIN3
- C13 pad 2: /ADS1299/AIN2P -> /ADS1299/REF
- C14 pad 1: /ADS1299/AIN3N -> /ADS1299/AIN2
- C14 pad 2: GND -> /ADS1299/REF
- C15 pad 1: GND -> /ADS1299/AIN1
- C15 pad 2: /ADS1299/AIN3P -> /ADS1299/REF
- C16 pad 1: /ADS1299/AIN4N -> /ADS1299 Power/+5V
- C16 pad 2: GND -> GNDD
- C17 pad 1: GND -> /ADS1299 Power/+3V3A
- C17 pad 2: /ADS1299/AIN4P -> GNDA
- C18 pad 1: /ADS1299/AIN6N -> /ADS1299 Power/-3V3A
- C18 pad 2: GND -> GNDA
- C19 pad 1: GND -> Net-(C19-Pad1)
- C19 pad 2: /ADS1299/AIN6P -> GNDA
- C2 pad 1: Net-(C2-Pad1) -> GND
- C2 pad 2: Net-(C2-Pad2) -> /Isolation/+3V3_ni
- C20 pad 1: /ADS1299/AIN5N -> /ADS1299 Power/+3V3
- C20 pad 2: GND -> GNDD
- C21 pad 1: GND -> Net-(C21-Pad1)
- C21 pad 2: /ADS1299/AIN5P -> GNDA
- C22 pad 1: /ADS1299/AIN7N -> Net-(C19-Pad1)
- C22 pad 2: GND -> GNDA
- C23 pad 1: GND -> Net-(C21-Pad1)
- C23 pad 2: /ADS1299/AIN7P -> GNDA
- C24 pad 1: /ADS1299/AIN8N -> /ADS1299 Power/+3V3A
- C24 pad 2: GND -> GNDA
- C25 pad 1: GND -> /ADS1299 Power/+2V5
- C25 pad 2: /ADS1299/AIN8P -> GNDA
- C3 pad 1: +3V3 -> GND
- C3 pad 2: GND -> /Isolation/+3V3_ni
- C4 pad 1: -3V3 -> GNDD
- C4 pad 2: GND -> /ADS1299 Power/+3V3
- C5 pad 1: +3V3 -> GNDD
- C5 pad 2: GND -> /ADS1299 Power/+3V3
- C6 pad 1: -3V3 -> GNDD
- C6 pad 2: GND -> /ADS1299 Power/+5V
- C7 pad 1: Net-(C7-Pad1) -> /ADS1299/AIN8
- C7 pad 2: GND -> /ADS1299/REF
- C8 pad 1: VDDA -> /ADS1299/AIN7
- C8 pad 2: GND -> /ADS1299/REF
- C9 pad 1: VSSA -> /ADS1299/AIN6
- C9 pad 2: GND -> /ADS1299/REF
- J1 pad 1: VSSA -> Net-(J1-Pad1)
- J1 pad 2: VSSA -> Net-(J1-Pad2)
- J1 pad 3: Net-(J1-Pad3) -> GND
- J2 pad 1: /nRF52840/nCS1 -> GND
- J2 pad 2: /nRF52840/MOSI -> /Isolation/+3V3_ni
- J2 pad 3: GND -> /nRF52840 Feather Sense Express Board/SDA_ni
- J2 pad 4: VDC -> /nRF52840 Feather Sense Express Board/SCL_ni
- R1 pad 1: /ADS1299/AIN1N -> Net-(R1-Pad1)
- R1 pad 2: /EEG-Electrodes/ELEC1N -> /nRF52840 Feather Sense Express Board/SD-nCS_ni
- R10 pad 1: /ADS1299/AIN6P -> /Isolation/+3V3_ni
- R10 pad 2: /EEG-Electrodes/ELEC6P -> Net-(R1-Pad1)
- R11 pad 1: /ADS1299/AIN5N -> /Isolation/+3V3_ni
- R11 pad 2: /EEG-Electrodes/ELEC5N -> Net-(R11-Pad2)
- R12 pad 1: /ADS1299/AIN5P -> /Isolation/+3V3_ni
- R12 pad 2: /EEG-Electrodes/ELEC5P -> Net-(R12-Pad2)
- R14 pad 1: /ADS1299/AIN7P -> /Isolation/MISO_ni
- R14 pad 2: /EEG-Electrodes/ELEC7P -> /Isolation/MISO_ni
- R15 pad 1: /ADS1299/AIN8N -> /Isolation/MOSI_ni
- R15 pad 2: /EEG-Electrodes/ELEC8N -> /Isolation/MOSI_ni
- R16 pad 1: /ADS1299/AIN8P -> /Isolation/SCK_ni
- R16 pad 2: /EEG-Electrodes/ELEC8P -> /Isolation/SCK_ni
- R17 pad 1: VDC -> Net-(C1-Pad2)
- R17 pad 2: /nRF52840/nCS0 -> /Isolation/+3V3_ni
- R18 pad 1: VDC -> GNDD
- R18 pad 2: /nRF52840/nCS1 -> Net-(D2-Pad1)
- R2 pad 1: /ADS1299/AIN1P -> Net-(R2-Pad1)
- R2 pad 2: /EEG-Electrodes/ELEC1P -> /nRF52840 Feather Sense Express Board/ADS-nDRDY_ni
- R3 pad 1: /ADS1299/AIN2N -> GND
- R3 pad 2: /EEG-Electrodes/ELEC2N -> Net-(D1-Pad1)
- R4 pad 1: /ADS1299/AIN2P -> Net-(R11-Pad2)
- R4 pad 2: /EEG-Electrodes/ELEC2P -> /nRF52840 Feather Sense Express Board/SD-nWP_ni
- R5 pad 1: /ADS1299/AIN3N -> Net-(R5-Pad1)
- R5 pad 2: /EEG-Electrodes/ELEC3N -> /nRF52840 Feather Sense Express Board/ADS-nRST_ni
- R6 pad 1: /ADS1299/AIN3P -> Net-(R12-Pad2)
- R6 pad 2: /EEG-Electrodes/ELEC3P -> /nRF52840 Feather Sense Express Board/SD-nCD_ni
- R7 pad 1: /ADS1299/AIN4N -> Net-(R7-Pad1)
- R7 pad 2: /EEG-Electrodes/ELEC4N -> /nRF52840 Feather Sense Express Board/ADS-nCS_ni
- R8 pad 1: /ADS1299/AIN4P -> /Isolation/+3V3_ni
- R8 pad 2: /EEG-Electrodes/ELEC4P -> Net-(R7-Pad1)
- R9 pad 1: /ADS1299/AIN6N -> /Isolation/+3V3_ni
- R9 pad 2: /EEG-Electrodes/ELEC6N -> Net-(R7-Pad1)
- U1 pad 1: /ADS1299/AIN8N -> Net-(U1-Pad1)
- U1 pad 10: /ADS1299/AIN4P -> Net-(U1-Pad10)
- U1 pad 11: /ADS1299/AIN3N -> /Isolation/SCK_ni
- U1 pad 12: /ADS1299/AIN3P -> /Isolation/MOSI_ni
- U1 pad 13: /ADS1299/AIN2N -> /Isolation/MISO_ni
- U1 pad 14: /ADS1299/AIN2P -> Net-(J1-Pad1)
- U1 pad 15: /ADS1299/AIN1N -> Net-(J1-Pad2)
- U1 pad 16: /ADS1299/AIN1P -> Net-(U1-Pad16)
- U1 pad 17: Net-(U1-Pad17) -> /nRF52840 Feather Sense Express Board/SDA_ni
- U1 pad 18: Net-(U1-Pad18) -> /nRF52840 Feather Sense Express Board/SCL_ni
- U1 pad 19: VDDA -> Net-(R12-Pad2)
- U1 pad 2: /ADS1299/AIN8P -> /Isolation/+3V3_ni
- U1 pad 20: VSSA -> Net-(R11-Pad2)
- U1 pad 21: VDDA -> Net-(R1-Pad1)
- U1 pad 22: VDDA -> Net-(R7-Pad1)
- U1 pad 23: VSSA -> Net-(R5-Pad1)
- U1 pad 24: Net-(U1-Pad24) -> Net-(R2-Pad1)
- U1 pad 27: (no net) -> Net-(U1-Pad27)
- U1 pad 3: /ADS1299/AIN7N -> Net-(U1-Pad3)
- U1 pad 4: /ADS1299/AIN7P -> GND
- U1 pad 5: /ADS1299/AIN6N -> Net-(U1-Pad5)
- U1 pad 6: /ADS1299/AIN6P -> Net-(U1-Pad6)
- U1 pad 7: /ADS1299/AIN5N -> Net-(U1-Pad7)
- U1 pad 8: /ADS1299/AIN5P -> Net-(U1-Pad8)
- U1 pad 9: /ADS1299/AIN4N -> Net-(U1-Pad9)
- U2 pad 1: Net-(U2-Pad1) -> /Isolation/+3V3_ni
- U2 pad 11: /nRF52840/SCK -> /ADS1299/SCK
- U2 pad 12: /nRF52840/MOSI -> /ADS1299/nCS
- U2 pad 13: /nRF52840/MISO -> /ADS1299/ADS_nRST
- U2 pad 14: Net-(U2-Pad14) -> /ADS1299/MOSI
- U2 pad 15: Net-(U2-Pad15) -> GNDD
- U2 pad 16: Net-(U2-Pad16) -> /ADS1299 Power/+3V3
- U2 pad 2: VDC -> GND
- U2 pad 3: Net-(U2-Pad3) -> /Isolation/MOSI_ni
- U2 pad 4: GND -> /nRF52840 Feather Sense Express Board/ADS-nRST_ni
- U2 pad 5: Net-(U2-Pad5) -> /nRF52840 Feather Sense Express Board/ADS-nCS_ni
- U2 pad 6: Net-(U2-Pad6) -> /Isolation/SCK_ni
- U2 pad 7: Net-(U2-Pad7) -> (no net)
- U2 pad 8: Net-(U2-Pad8) -> GND
- U2 pad 9: Net-(U2-Pad9) -> GNDD
- U3 pad 1: VDC -> /ADS1299 Power/+3V3
- U3 pad 2: GND -> GNDD
- U3 pad 3: Net-(U3-Pad3) -> /ADS1299/MISO
- U3 pad 4: Net-(U3-Pad4) -> /ADS1299/ADS_nDRDY
- U3 pad 5: +3V3 -> Net-(U3-Pad5)
- U4 pad 2: Net-(C2-Pad1) -> GND
- U4 pad 5: -3V3 -> GNDD
- U4 pad 6: Net-(U4-Pad6) -> (no net)
- U4 pad 7: Net-(U4-Pad7) -> /ADS1299 Power/+5V
- U5 pad 1: +3V3 -> /ADS1299 Power/+5V
- U5 pad 2: GND -> GNDD
- U5 pad 3: +3V3 -> /ADS1299 Power/+5V
- U5 pad 4: Net-(U5-Pad4) -> (no net)
- U5 pad 5: VDDA -> /ADS1299 Power/+3V3
- U6 pad 1: GND -> Net-(C19-Pad1)
- U6 pad 2: -3V3 -> Net-(C19-Pad1)
- U6 pad 3: -3V3 -> (no net)
- U6 pad 4: Net-(C7-Pad1) -> /ADS1299 Power/-3V3A
- U6 pad 5: VSSA -> (no net)
- U7 pad 1: Net-(U7-Pad1) -> /ADS1299 Power/+3V3A
- U7 pad 2: /nRF52840/MOSI -> GNDA
- U7 pad 3: /nRF52840/ADS-nRST -> /ADS1299 Power/+3V3A
- U7 pad 4: /nRF52840/nCS0 -> (no net)
- U7 pad 5: /nRF52840/SCK -> Net-(C21-Pad1)
- U8 pad 3: Net-(U8-Pad3) -> GNDA
- U8 pad 6: Net-(U8-Pad6) -> Net-(JP2-Pad1)
- U8 pad 7: Net-(U8-Pad6) -> Net-(U8-Pad7)
- U8 pad 8: Net-(U8-Pad6) -> /ADS1299 Power/+3V3A
Routing:
- net /Isolation/+3V3_ni: track 0.00 -> 41.0 mm, vias 0 -> 1
- net GNDD: track 0.00 -> 14.2 mm, vias 0 -> 2
- net /ADS1299 Power/+3V3: track 0.00 -> 14.1 mm
- net GND: track 0.00 -> 12.1 mm, vias 0 -> 4
- net /ADS1299 Power/+5V: track 0.00 -> 4.81 mm
- net /nRF52840 Feather Sense Express Board/ADS-nRST_ni: track 0.00 -> 4.00 mm, vias 0 -> 1
- net /nRF52840 Feather Sense Express Board/ADS-nCS_ni: track 0.00 -> 4.00 mm, vias 0 -> 1
- net /Isolation/MISO_ni: track 0.00 -> 4.00 mm, vias 0 -> 1
- net Net-(JP5-Pad2): track 0.00 -> 3.92 mm
- net Net-(JP4-Pad1): track 0.00 -> 2.85 mm
- net Net-(JP3-Pad2): track 0.00 -> 2.83 mm
- net /nRF52840 Feather Sense Express Board/ADS-nDRDY_ni: track 0.00 -> 2.00 mm, vias 0 -> 1
- net /Isolation/SCK_ni: track 0.00 -> 2.00 mm, vias 0 -> 1
- net /Isolation/MOSI_ni: track 0.00 -> 2.00 mm, vias 0 -> 1
- added copper zone on B.Cu, net GND
- added copper zone on B.Cu, net GNDD
Other:
- board outline removed

Commit message: Layout of the NRF52840 section of the PCB.
Parts:
- moved R3 406.5 mm to (2.21, 199.9), turned to 180 degrees
- moved R16 394.0 mm to (2.48, 165.9), turned to 270 degrees
- moved C46 381.5 mm to (27.5, 88.0)
- moved C47 381.5 mm to (19.1, 90.2)
- moved C55 381.5 mm to (13.9, 91.1)
- moved R32 381.5 mm to (40.8, 88.3)
- moved C42 381.5 mm to (39.1, 83.3)
- moved C43 381.5 mm to (39.1, 80.8)
- moved C44 381.5 mm to (27.8, 90.5)
- moved C45 381.5 mm to (34.7, 83.3)
- moved C48 381.5 mm to (34.7, 80.8)
- moved C49 381.5 mm to (34.7, 75.8)
- moved C50 381.5 mm to (23.4, 90.5)
- moved C51 381.5 mm to (39.1, 75.8)
- moved C52 381.5 mm to (34.7, 78.3)
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Connections:
- R1 pad 2: /nRF52840 Feather Sense Express Board/SD-nCS_ni -> /nRF52840 Feather Sense Express Board/SD-nWP_ni
- R14 pad 2: /Isolation/MISO_ni -> Net-(R14-Pad2)
- R15 pad 2: /Isolation/MOSI_ni -> Net-(R15-Pad2)
- R16 pad 2: /Isolation/SCK_ni -> Net-(R16-Pad2)
- R4 pad 2: /nRF52840 Feather Sense Express Board/SD-nWP_ni -> /nRF52840 Feather Sense Express Board/SD-nCD_ni
- R6 pad 2: /nRF52840 Feather Sense Express Board/SD-nCD_ni -> /nRF52840 Feather Sense Express Board/SD-nCS_ni
- R8 pad 2: Net-(R7-Pad1) -> Net-(R5-Pad1)
- TP1 pad 1: /nRF52840 Feather Sense Express Board/SD-nCD_ni -> /nRF52840 Feather Sense Express Board/SD-nCS_ni
- TP2 pad 1: /nRF52840 Feather Sense Express Board/SD-nWP_ni -> /nRF52840 Feather Sense Express Board/SD-nCD_ni
- TP3 pad 1: /nRF52840 Feather Sense Express Board/SD-nCS_ni -> /nRF52840 Feather Sense Express Board/SD-nWP_ni
- U1 pad 11: /Isolation/SCK_ni -> Net-(R16-Pad2)
- U1 pad 12: /Isolation/MOSI_ni -> Net-(R15-Pad2)
- U1 pad 13: /Isolation/MISO_ni -> Net-(R14-Pad2)
Routing:
- net /nRF52840 Feather Sense Express Board/SD-nWP_ni: track 0.00 -> 72.2 mm, vias 0 -> 2
- net /nRF52840 Feather Sense Express Board/SD-nCD_ni: track 0.00 -> 56.6 mm, vias 0 -> 2
- net /nRF52840 Feather Sense Express Board/SDA_ni: track 0.00 -> 48.0 mm
- net /nRF52840 Feather Sense Express Board/SD-nCS_ni: track 0.00 -> 47.3 mm, vias 0 -> 2
- net /Isolation/MISO_ni: track 4.00 -> 48.3 mm
- net /nRF52840 Feather Sense Express Board/SCL_ni: track 0.00 -> 40.5 mm
- net /nRF52840 Feather Sense Express Board/ADS-nDRDY_ni: track 2.00 -> 40.7 mm
- net Net-(R16-Pad2): track 0.00 -> 38.2 mm
- net Net-(R15-Pad2): track 0.00 -> 38.0 mm
- net Net-(R14-Pad2): track 0.00 -> 37.8 mm
- net /Isolation/SCK_ni: track 2.00 -> 37.5 mm
- net /Isolation/MOSI_ni: track 2.00 -> 33.6 mm
- net /nRF52840 Feather Sense Express Board/ADS-nCS_ni: track 4.00 -> 30.6 mm, vias 1 -> 2
- net GND: track 12.1 -> 38.7 mm, vias 4 -> 5
- net /nRF52840 Feather Sense Express Board/ADS-nRST_ni: track 4.00 -> 30.0 mm, vias 1 -> 2
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- removed copper zone on B.Cu, net GND
- removed copper zone on B.Cu, net GNDD

Commit message: Further PCB Layout.
Parts:
- U6: footprint Package_CSP:LFCSP-8-1EP_3x3mm_P0.5mm_EP1.45x1.74mm -> Package_TO_SOT_SMD:TSOT-23-5
- moved C40 120.3 mm to (-22.1, 71.1)
- moved C38 119.0 mm to (-22.4, 74.6)
- moved TP30 115.4 mm to (24.6, 112.8)
- moved C31 112.9 mm to (-17.1, 59.2)
- moved C33 111.0 mm to (-17.0, 61.7)
- moved C39 107.8 mm to (28.5, 122.1), turned to 90 degrees
- moved L4 106.9 mm to (25.5, 123.0)
- moved C41 106.8 mm to (25.5, 121.0)
- moved C35 106.0 mm to (-9.40, 48.1)
- moved C36 106.0 mm to (-14.0, 48.5)
- moved C37 104.9 mm to (30.5, 122.1), turned to 90 degrees
- moved C30 104.6 mm to (33.8, 115.5), turned to 180 degrees
- moved U8 102.8 mm to (34.5, 120.5), turned to 270 degrees
- moved JP2 101.4 mm to (31.4, 126.0), turned to 180 degrees
- moved JP1 100.1 mm to (39.1, 115.6), turned to 0 degrees
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Connections:
- U6 pad 1: Net-(C19-Pad1) -> GNDA
- U6 pad 2: Net-(C19-Pad1) -> /ADS1299 Power/-3V3A
- U6 pad 3: (no net) -> /ADS1299 Power/-3V3A
- U6 pad 4: /ADS1299 Power/-3V3A -> Net-(U6-Pad4)
- U6 pad 5: (no net) -> Net-(C19-Pad1)
Routing:
- net GNDA: track 0.00 -> 53.6 mm, vias 0 -> 5
- net /ADS1299 Power/-2V5: track 0.00 -> 27.6 mm, vias 0 -> 3
- net /ADS1299 Power/+3V3A: track 0.00 -> 17.5 mm, vias 0 -> 2
- net /ADS1299 Power/+5V: track 4.81 -> 16.0 mm
- net GNDD: track 14.2 -> 24.0 mm
- net Net-(C52-Pad1): track 0.00 -> 8.42 mm
- net Net-(C21-Pad1): track 0.00 -> 6.35 mm
- net Net-(C37-Pad1): track 0.00 -> 6.11 mm
- net Net-(C19-Pad1): track 0.00 -> 6.02 mm
- net /ADS1299 Power/+2V5: track 0.00 -> 5.67 mm
- net Net-(C42-Pad2): track 0.00 -> 5.33 mm
- net /ADS1299 Power/-3V3A: track 0.00 -> 5.24 mm
- net Net-(C54-Pad1): track 0.00 -> 4.47 mm
- net Net-(JP2-Pad1): track 0.00 -> 4.38 mm
- net /ADS1299 Power/+3V3: track 14.1 -> 18.3 mm
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