File: hardware/DevBoard/DevBoard.kicad_sch (KiCad schematic)
At the start: 8 parts, among them J1 Conn_02x06_Odd_Even, J2 Conn_02x06_Odd_Even, J3 Conn_02x01, J4 Conn_01x10, J5 Conn_01x07, U1 Adafruit_SD_Breakout, U2 nRF52840-Feather-Sense

Commit message: Updates
WIP
Parts:
- added J6: Conn_02x06_Odd_Even, VolksEEG:6-Jumper Header, symbol Connector_Generic:Conn_02x06_Odd_Even
- added SW1, SW2, SW3, SW4, SW5: Tact-Switch, VolksEEG:Sparkfun Tactile Switch, symbol VolksEEG:Tact-Switch
- added SW6: Reset Switch, VolksEEG:Sparkfun Tactile Switch, symbol VolksEEG:Tact-Switch
- added U4: Adafruit-4650-FeatherWing-128x64, VolksEEG:nRF52840_Feather_Sense, symbol VolksEEG:Adafruit-4650-FeatherWing-128x64
- U3: value (none) -> ADS1299EEGFE-PDK; footprint (none) -> VolksEEG:ADS1299EEGFE-PDK
Connections:
- net 3V3_nrf: now also U4.2 (3V)
- net A0_nrf: now also J6.8 (Pin_8)
- net A1_nrf: now also J6.10 (Pin_10)
- net A2_nrf: now also J6.12 (Pin_12)
- net GND: now also SW1.1, SW1.2, SW2.1, SW2.2, SW3.1, SW3.2, SW4.1, SW4.2, SW5.1, SW5.2, SW6.1, SW6.2
- net GND_nrf: now also U4.4 (GND)
- net GPIO11_nrf: now also J6.4 (Pin_4)
- net GPIO13_nrf: now also J6.6 (Pin_6)
- net GPIO6_nrf: now also J6.2 (Pin_2)
- net MISO: no longer U1.5 (D_Out)
- net MISO_nrf: now also U1.5 (D_Out)
- net MOSI: no longer U1.6 (D_in)
- net MOSI_nrf: now also U1.6 (D_in)
- net RST_nrf: now also SW6.3 (K), SW6.4 (A), U4.1 (RST)
- net SCK: no longer U1.4 (CLK)
- net SCK_nrf: now also U1.4 (CLK)
- net SCL_nrf: now also U4.18 (SCL)
- net SDA_nrf: now also U4.17 (SDA)
- net ~{CARD_CD_nrf}: now also U1.8 (Card_Detect)
- net ~{CARD_CS_nrf}: now also U1.7 (~{Chip_Select})
- net ~{CD_sdc}: no longer U1.8 (Card_Detect)
- net ~{CS_sdc}: no longer U1.7 (~{Chip_Select})
- new net sw1: J6.1 (Pin_1)
- new net sw2: J6.3 (Pin_3), SW2.3 (K), SW2.4 (A)
- new net sw3: J6.5 (Pin_5), SW3.3 (K), SW3.4 (A)
- new net sw4: J6.7 (Pin_7), SW4.3 (K), SW4.4 (A)
- new net sw5: J6.9 (Pin_9), SW5.3 (K), SW5.4 (A)
- new net sw6: J6.11 (Pin_11)
- new net sw_a: SW1.3, SW1.4
Other:
- moved on the sheet: J1, J2, J3, J4, J5, U2, U3
