File: hardware/DevBoard/DevBoard.kicad_sch (KiCad schematic)
At the start: 16 parts, among them J1 Conn_02x06_Odd_Even, J2 Conn_02x06_Odd_Even, J3 Conn_02x01, J4 Conn_01x10, J5 Conn_01x07, J6 Conn_02x06_Odd_Even, SW1 Tact-Switch, SW2 Tact-Switch, SW3 Tact-Switch, SW4 Tact-Switch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

Commit message: As sent to JLBPC
Parts:
- U3: value (none) -> ADS1299EEGFE-PDK
Connections:
- net SW1_nrf is gone; now on net GPIO6_nrf: J6.2 (Pin_2), U2.20 (6)
- net SW2_nrf is gone; now on net GPIO11_nrf: J6.4 (Pin_4), U2.23 (11)
- net SW3_nrf is gone; now on net GPIO13_nrf: J6.6 (Pin_6), U2.25 (13)
- net sw_a is gone; now on net sw1: SW1.3, SW1.4
- net A2_nrf: no longer J6.12 (Pin_12)
- net RST_nrf: now also J6.12 (Pin_12); no longer SW6.3, SW6.4
- net sw6: now also SW6.3, SW6.4
Changed lines of the file:
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@@
     (company "VolksEEG Project")
     (comment 1 "Or by reading files from EDF file on SD card")
-    (comment 2 "Can be used using TI ADS1299 Dev board for live data")
+    (comment 2 "Can be used with TI ADS1299 Dev board for live data")
   )
   (junction (at 147.32 90.17) (diameter 0) (color 0 0 0 0)
@@
     (effects (font (size 1.27 1.27)) (justify left bottom))
   )
-  (label "SW1_nrf" (at 140.97 111.76 0)
-    (effects (font (size 1.27 1.27)) (justify left bottom))
-  )
-  (label "sw_a" (at 125.73 44.45 0)
+  (label "GPIO6_nrf" (at 140.97 111.76 0)
+    (effects (font (size 1.27 1.27)) (justify left bottom))
+  )
+  (label "sw1" (at 125.73 44.45 0)
     (effects (font (size 1.27 1.27)) (justify left bottom))
   )
@@
     (effects (font (size 1.27 1.27)) (justify left bottom))
   )
-  (label "SW2_nrf" (at 140.97 114.3 0)
+  (label "GPIO11_nrf" (at 140.97 114.3 0)
     (effects (font (size 1.27 1.27)) (justify left bottom))
   )
@@
     (effects (font (size 1.27 1.27)) (justify left bottom))
   )
-  (label "SW2_nrf" (at 34.29 114.3 0)
+  (label "GPIO11_nrf" (at 34.29 114.3 0)
     (effects (font (size 1.27 1.27)) (justify left bottom))
   )
@@
     (effects (font (size 1.27 1.27)) (justify left bottom))
   )
-  (label "SW1_nrf" (at 34.29 106.68 0)
+  (label "GPIO6_nrf" (at 34.29 106.68 0)
     (effects (font (size 1.27 1.27)) (justify left bottom))
   )
@@
     (effects (font (size 1.27 1.27)) (justify left bottom))
   )
-  (label "A2_nrf" (at 140.97 124.46 0)
+  (label "RST_nrf" (at 140.97 124.46 0)
     (effects (font (size 1.27 1.27)) (justify left bottom))
   )
@@
     (effects (font (size 1.27 1.27)) (justify left bottom))
   )
-  (label "RST_nrf" (at 160.02 87.63 0)
+  (label "sw6" (at 160.02 87.63 0)
     (effects (font (size 1.27 1.27)) (justify left bottom))
   )
@@
     (effects (font (size 1.27 1.27)) (justify left bottom))
   )
-  (label "SW3_nrf" (at 140.97 116.84 0)
+  (label "GPIO13_nrf" (at 140.97 116.84 0)
     (effects (font (size 1.27 1.27)) (justify left bottom))
   )
@@
     (effects (font (size 1.27 1.27)) (justify left bottom))
   )
-  (label "SW3_nrf" (at 34.29 119.38 0)
+  (label "GPIO13_nrf" (at 34.29 119.38 0)
     (effects (font (size 1.27 1.27)) (justify left bottom))
   )
@@
     (in_bom yes) (on_board yes) (fields_autoplaced)
     (property "Reference" "U3" (id 0) (at 208.28 26.67 0))
-    (property "Value" "" (id 1) (at 208.28 29.21 0))
+    (property "Value" "ADS1299EEGFE-PDK" (id 1) (at 208.28 29.21 0))
     (property "Footprint" "VolksEEG:ADS1299EEGFE-PDK" (id 2) (at 227.33 49.53 0)
       (effects (font (size 1.27 1.27)) hide)
